File: Hardware/ECU/Crank-and-Cam.kicad_sch (KiCad schematic)
At the start: 21 parts, among them IC1 MAX9926UAEE_V+, Q1 Q_DUAL_NMOS_S1G1D2S2G2D1, SW1 SW_DPDT_x2, SW2 SW_DPDT_x2, SW3 SW_DIP_x02

Commit message: PCB v0.3
Ready to Build
Parts:
- removed SW3: SW_DIP_x02, Button_Switch_SMD:SW_DIP_SPSTx02_Slide_9.78x7.26mm_W8.61mm_P2.54mm, symbol Switch:SW_DIP_x02
- added JP1, JP5: Jumper_2_Open, Jumper:SolderJumper-2_P1.3mm_Open_Pad1.0x1.5mm, symbol Jumper:Jumper_2_Open
Connections:
- net MCU-D19: now also JP1.1 (A), JP5.1 (A)
- net at C5.1: now also JP5.2 (B)
- net at C4.2: now also JP1.2 (B)
Changed lines of the file:
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@@
 	(wire
 		(pts
-			(xy 120.65 83.82) (xy 128.27 83.82)
+			(xy 107.95 83.82) (xy 118.11 83.82)
 		)
 		(stroke
@@
 	(wire
 		(pts
+			(xy 118.11 68.58) (xy 118.11 71.12)
+		)
+		(stroke
+			(width 0)
+			(type default)
+		)
+	)
+	(wire
+		(pts
 			(xy 53.34 101.6) (xy 53.34 105.41)
 		)
@@
 	(wire
 		(pts
-			(xy 53.34 81.28) (xy 53.34 77.47)
+			(xy 120.65 83.82) (xy 128.27 83.82)
 		)
 		(stroke
@@
 	(wire
 		(pts
-			(xy 242.57 83.82) (xy 223.52 83.82)
+			(xy 53.34 81.28) (xy 53.34 77.47)
 		)
 		(stroke
@@
 	(wire
 		(pts
-			(xy 223.52 93.98) (xy 218.44 93.98)
+			(xy 242.57 83.82) (xy 223.52 83.82)
 		)
 		(stroke
@@
 	(wire
 		(pts
-			(xy 223.52 96.52) (xy 215.9 96.52)
+			(xy 223.52 93.98) (xy 218.44 93.98)
 		)
 		(stroke
@@
 	(wire
 		(pts
-			(xy 77.47 105.41) (xy 87.63 105.41)
+			(xy 223.52 96.52) (xy 215.9 96.52)
 		)
 		(stroke
@@
 	(wire
 		(pts
-			(xy 231.14 86.36) (xy 223.52 86.36)
+			(xy 77.47 105.41) (xy 87.63 105.41)
 		)
 		(stroke
@@
 	(wire
 		(pts
-			(xy 107.95 83.82) (xy 118.11 83.82)
+			(xy 231.14 86.36) (xy 223.52 86.36)
 		)
 		(stroke
@@
 	(wire
 		(pts
+			(xy 120.65 81.28) (xy 120.65 83.82)
+		)
+		(stroke
+			(width 0)
+			(type default)
+		)
+	)
+	(wire
+		(pts
 			(xy 218.44 93.98) (xy 215.9 93.98)
 		)
@@
 	(wire
 		(pts
+			(xy 120.65 68.58) (xy 120.65 71.12)
+		)
+		(stroke
+			(width 0)
+			(type default)
+		)
+	)
+	(wire
+		(pts
 			(xy 96.52 72.39) (xy 96.52 73.66)
 		)
@@
 	(wire
 		(pts
+			(xy 118.11 81.28) (xy 118.11 83.82)
+		)
+		(stroke
+			(width 0)
+			(type default)
+		)
+	)
+	(wire
+		(pts
 			(xy 106.68 99.06) (xy 113.03 99.06)
 		)
@@
 	)
 	(symbol
+		(lib_id "Jumper:Jumper_2_Open")
+		(at 120.65 76.2 270)
+		(mirror x)
+		(unit 1)
+		(exclude_from_sim no)
+		(in_bom yes)
+		(on_board yes)
+		(dnp no)
+		(property "Reference" "JP5"
+			(at 126.619 76.2 0)
+			(effects
+				(font
+					(size 1.27 1.27)
+				)
+			)
+		)
+		(property "Value" "Jumper_2_Open"
+			(at 124.3076 76.2 0)
+			(effects
+				(font
+					(size 1.27 1.27)
+				)
+			)
+		)
+		(property "Footprint" "Jumper:SolderJumper-2_P1.3mm_Open_Pad1.0x1.5mm"
+			(at 120.65 76.2 0)
+			(effects
+				(font
+					(size 1.27 1.27)
+				)
+				(hide yes)
+			)
+		)
+		(property "Datasheet" "~"
+			(at 120.65 76.2 0)
+			(effects
+				(font
+					(size 1.27 1.27)
+				)
+				(hide yes)
+			)
+		)
+		(property "Description" ""
+			(at 120.65 76.2 0)
+			(effects
+				(font
+					(size 1.27 1.27)
+				)
+				(hide yes)
+			)
+		)
+		(pin "1"
+		)
+		(pin "2"
+		)
+		(instances
+			(project "ECU"
+				(path "/aaebd8f9-fdac-426b-87c0-a208167b6035/34d8184b-485a-4241-8a68-5c8e24cc7ad9"
+					(reference "JP5")
+					(unit 1)
+				)
+			)
+		)
+	)
+	(symbol
 		(lib_id "Device:R")
 		(at 100.33 80.01 180)
@@
 	)
 	(symbol
-		(lib_id "Switch:SW_DIP_x02")
-		(at 118.11 76.2 270)
-		(unit 1)
-		(exclude_from_sim no)
-		(in_bom yes)
-		(on_board yes)
-		(dnp no)
-		(property "Reference" "SW3"
-			(at 123.952 75.0316 90)
-			(effects
-				(font
-					(size 1.27 1.27)
-				)
-				(justify left)
-			)
-		)
-		(property "Value" "SW_DIP_x02"
-			(at 123.952 77.343 90)
-			(effects
-				(font
-					(size 1.27 1.27)
-				)
-				(justify left)
-			)
-		)
-		(property "Footprint" "Button_Switch_SMD:SW_DIP_SPSTx02_Slide_9.78x7.26mm_W8.61mm_P2.54mm"
-			(at 123.952 78.5114 90)
-			(effects
-				(font
-					(size 1.27 1.27)
-				)
-				(justify left)
-				(hide yes)
-			)
-		)
-		(property "Datasheet" "~"
-			(at 118.11 76.2 0)
-			(effects
-				(font
-					(size 1.27 1.27)
-				)
-				(hide yes)
-			)
-		)
-		(property "Description" ""
-			(at 118.11 76.2 0)
-			(effects
-				(font
-					(size 1.27 1.27)
-				)
-				(hide yes)
-			)
-		)
-		(property "Digikey Part Number" "679-3566-1-ND"
-			(at 118.11 76.2 0)
-			(effects
-				(font
-					(size 1.27 1.27)
-				)
-				(hide yes)
-			)
-		)
-		(property "Manufacturer_Name" "APEM Inc."
-			(at 118.11 76.2 0)
-			(effects
-				(font
-					(size 1.27 1.27)
-				)
-				(hide yes)
-			)
-		)
-		(property "Manufacturer_Part_Number" "IKN0204000"
-			(at 118.11 76.2 0)
-			(effects
-				(font
-					(size 1.27 1.27)
-				)
-				(hide yes)
-			)
-		)
-		(property "URL" "https://www.digikey.com.au/product-detail/en/apem-inc/IKN0204000/679-3566-1-ND/4384369"
-			(at 118.11 76.2 0)
-			(effects
-				(font
-					(size 1.27 1.27)
-				)
-				(hide yes)
-			)
-		)
-		(pin "1"
-		)
-		(pin "2"
-		)
-		(pin "3"
-		)
-		(pin "4"
-		)
-		(instances
-			(project "ECU"
-				(path "/aaebd8f9-fdac-426b-87c0-a208167b6035/34d8184b-485a-4241-8a68-5c8e24cc7ad9"
-					(reference "SW3")
-					(unit 1)
-				)
-			)
-		)
-	)
-	(symbol
 		(lib_id "Device:R")
 		(at 246.38 96.52 270)
@@
 					(unit 1)
 				)
+			)
+		)
+	)
+	(symbol
+		(lib_id "Jumper:Jumper_2_Open")
+		(at 118.11 76.2 90)
+		(unit 1)
+		(exclude_from_sim no)
+		(in_bom yes)
+		(on_board yes)
+		(dnp no)
+		(property "Reference" "JP1"
+			(at 112.141 76.2 0)
+			(effects
+				(font
+					(size 1.27 1.27)
+				)
+			)
+		)
+		(property "Value" "Jumper_2_Open"
+			(at 114.4524 76.2 0)
+			(effects
+				(font
+					(size 1.27 1.27)
+				)
+			)
+		)
+		(property "Footprint" "Jumper:SolderJumper-2_P1.3mm_Open_Pad1.0x1.5mm"
+			(at 118.11 76.2 0)
+			(effects
+				(font
+					(size 1.27 1.27)
+				)
+				(hide yes)
+			)
+		)
+		(property "Datasheet" "~"
+			(at 118.11 76.2 0)
+			(effects
+				(font
+					(size 1.27 1.27)
+				)
+				(hide yes)
+			)
+		)
+		(property "Description" ""
+			(at 118.11 76.2 0)
+			(effects
+				(font
+					(size 1.27 1.27)
+				)
+				(hide yes)
+			)
+		)
+		(pin "1"
+		)
+		(pin "2"
+		)
+		(instances
+			(project "ECU"
+				(path "/aaebd8f9-fdac-426b-87c0-a208167b6035/34d8184b-485a-4241-8a68-5c8e24cc7ad9"
+					(reference "JP1")
+					(unit 1)
+				)
