File: Hardware/ECU/ECU.kicad_pcb (KiCad board)
At the start: 2 copper layers, 148 x 111.5 mm, 161 parts, among them IC1 MAX9926UAEE_V+, IC2 ZXMS6006DT8, IC3 ZXMS6006DT8, IC4 ZXMS6006DT8, J1 Conn_01x04, Q1 Q_DUAL_NMOS_S1G1D2S2G2D1, Q2 Q_DUAL_NMOS_S1G1D2S2G2D1, Q3 Q_PNP_BCEC, Q4 IRFB4110PBF, Q5 IRFB4110PBF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

Commit message: PCB v0.3
Ready to Build
Parts:
- removed SW3: SW_DIP_x02, Button_Switch_SMD:SW_DIP_SPSTx02_Slide_9.78x7.26mm_W8.61mm_P2.54mm
- added JP1: Jumper_2_Open, Jumper:SolderJumper-2_P1.3mm_Open_Pad1.0x1.5mm, F.Cu at (75.7, 134.7)
- added JP5: Jumper_2_Open, Jumper:SolderJumper-2_P1.3mm_Open_Pad1.0x1.5mm, F.Cu at (72.6, 134.7)
- moved C5 0.13 mm to (72.6, 139.3)
- moved C4 0.08 mm to (75.7, 139.3)
Routing:
- net MCU-A5: track 129.9 -> 138.4 mm
- net Net-(JP1-B): track 3.79 -> 3.00 mm
- net Net-(JP5-B): track 3.79 -> 3.00 mm
