File: Hardware/ECU/ECU.kicad_pcb (KiCad board)
At the start: 2 copper layers, 148 x 111.5 mm, 162 parts, among them IC1 MAX9926UAEE_V+, IC2 ZXMS6006DT8, IC3 ZXMS6006DT8, IC4 ZXMS6006DT8, J1 Conn_01x04, Q1 Q_DUAL_NMOS_S1G1D2S2G2D1, Q2 Q_DUAL_NMOS_S1G1D2S2G2D1, Q3 Q_PNP_BCEC, Q4 IRFB4110PBF, Q5 IRFB4110PBF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

Commit message: deleted:    Hardware/ECU/ECU-backups/ECU-2025-05-17_134922.zip deleted:    Hardware/ECU/ECU-backups/ECU-2025-05-18_153853.zip deleted:    Hardware/ECU/ECU-backups/ECU-2025-05-18_155339.zip 	deleted:    Hardware/ECU/ECU-backups/ECU-2025-05-18_160128.zip 	deleted:    Hardware/ECU/ECU-backups/ECU-2025-05-18_161219.zip 	deleted:    Hardware/ECU/ECU-backups/ECU-2025-05-18_185910.zip 	deleted:    Hardware/ECU/ECU-backups/ECU-2025-05-19_140656.zip 	deleted:    Hardware/ECU/ECU-backups/ECU-2025-05-19_142320.zip 	deleted:    Hardware/ECU/ECU-backups/ECU-2025-05-19_145225.zip 	deleted:    Hardware/ECU/ECU-backups/ECU-2025-05-19_160311.zip 	deleted:    Hardware/ECU/ECU-backups/ECU-2025-05-19_220542.zip 	deleted:    Hardware/ECU/ECU-backups/ECU-2025-05-20_084251.zip 	new file:   Hardware/ECU/ECU-backups/ECU-2025-06-18_111329.zip 	renamed:    Hardware/ECU/ECU-backups/ECU-2025-05-20_085713.zip -> Hardware/ECU/ECU-backups/ECU-2025-06-18_112509.zip 	renamed:    Hardware/ECU/ECU-backups/ECU-2025-05-20_090304.zip -> Hardware/ECU/ECU-backups/ECU-2025-06-18_114215.zip 	new file:   Hardware/ECU/ECU-backups/ECU-2025-06-18_151410.zip 	new file:   Hardware/ECU/ECU-backups/ECU-2025-06-18_152336.zip 	new file:   Hardware/ECU/ECU-backups/ECU-2025-06-23_105455.zip 	new file:   Hardware/ECU/ECU-backups/ECU-2025-06-23_135936.zip 	new file:   Hardware/ECU/ECU-backups/ECU-2025-06-23_145648.zip 	new file:   Hardware/ECU/ECU-backups/ECU-2025-06-23_161930.zip 	new file:   Hardware/ECU/ECU-backups/ECU-2025-06-23_163830.zip 	new file:   Hardware/ECU/ECU-backups/ECU-2025-06-25_140659.zip 	new file:   Hardware/ECU/ECU-backups/ECU-2025-06-25_142923.zip 	new file:   Hardware/ECU/ECU-backups/ECU-2025-06-25_144402.zip 	new file:   Hardware/ECU/ECU-backups/ECU-2025-06-25_155601.zip 	modified:   Hardware/ECU/ECU.kicad_pcb 	modified:   Hardware/ECU/ECU.kicad_prl 	new file:   Hardware/ECU/output/ECU-B_Cu.dxf 	new file:   Hardware/ECU/output/ECU-B_Cu.svg 	new file:   Hardware/ECU/output/ECU-F_Adhesive.dxf 	new fi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
Routing:
- net GND: track 1208.9 -> 1206.3 mm, vias 36 -> 48
- added copper zone on B.Cu, net GND
- added copper zone on F.Cu, net GND
Changed lines of the file:
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@@
 		(tenting front back)
 		(pcbplotparams
-			(layerselection 0x00000000_00000000_55555555_5755f5ff)
-			(plot_on_all_layers_selection 0x00000000_00000000_00000000_00000000)
+			(layerselection 0x00000000_00000000_55555555_55555555)
+			(plot_on_all_layers_selection 0x00000000_00000000_00000800_02000000)
 			(disableapertmacros no)
 			(usegerberextensions no)
@@
 			(dashed_line_dash_ratio 12.000000)
 			(dashed_line_gap_ratio 3.000000)
-			(svgprecision 4)
+			(svgprecision 6)
 			(plotframeref no)
 			(mode 1)
@@
 			(crossoutdnponfab yes)
 			(subtractmaskfromsilk no)
-			(outputformat 4)
+			(outputformat 5)
 			(mirror no)
-			(drillshape 2)
+			(drillshape 0)
 			(scaleselection 1)
 			(outputdirectory "output/")
@@
 	)
 	(gr_circle
-		(center 213 32)
-		(end 214 32)
+		(center 70 35.5)
+		(end 70.3 35.5)
 		(stroke
 			(width 0.1)
-			(type default)
-		)
-		(fill no)
-		(layer "User.3")
-	)
-	(gr_circle
-		(center 65 32)
-		(end 65 33)
-		(stroke
-			(width 0.1)
-			(type default)
-		)
-		(fill no)
-		(layer "User.3")
-	)
-	(gr_circle
-		(center 65 143.5)
-		(end 66 143.5)
-		(stroke
-			(width 0.1)
-			(type default)
+			(type solid)
 		)
-		(fill no)
+		(fill yes)
+		(locked yes)
 		(layer "User.3")
 	)
 	(gr_circle
-		(center 213 143.5)
-		(end 214 143.5)
+		(center 206 140.5)
+		(end 206.3 140.5)
 		(stroke
 			(width 0.1)
-			(type default)
+			(type solid)
 		)
-		(fill no)
+		(fill yes)
+		(locked yes)
 		(layer "User.3")
 	)
@@
 	)
 	(via
+		(at 141.9 90.2)
+		(size 0.6)
+		(drill 0.3)
+		(layers "F.Cu" "B.Cu")
+		(free yes)
+		(net 9)
+	)
+	(via
 		(at 119.5 49)
 		(size 0.6)
@@
 	)
 	(via
+		(at 138.1 140)
+		(size 0.6)
+		(drill 0.3)
+		(layers "F.Cu" "B.Cu")
+		(net 9)
+	)
+	(via
 		(at 151.985 112.985)
 		(size 0.6)
@@
 	)
 	(via
+		(at 164.6 93.9)
+		(size 0.6)
+		(drill 0.3)
+		(layers "F.Cu" "B.Cu")
+		(free yes)
+		(net 9)
+	)
+	(via
 		(at 203 100)
 		(size 0.6)
@@
 	)
 	(via
+		(at 83.9 114.6)
+		(size 0.6)
+		(drill 0.3)
+		(layers "F.Cu" "B.Cu")
+		(net 9)
+	)
+	(via
 		(at 199.5 77)
 		(size 0.6)
@@
 	)
 	(via
+		(at 150.5 96.1)
+		(size 0.6)
+		(drill 0.3)
+		(layers "F.Cu" "B.Cu")
+		(free yes)
+		(net 9)
+	)
+	(via
+		(at 136.7 134.2)
+		(size 0.6)
+		(drill 0.3)
+		(layers "F.Cu" "B.Cu")
+		(net 9)
+	)
+	(via
 		(at 108.5 122.5)
 		(size 0.6)
@@
 	)
 	(via
+		(at 157.5 118.5)
+		(size 0.6)
+		(drill 0.3)
+		(layers "F.Cu" "B.Cu")
+		(free yes)
+		(net 9)
+	)
+	(via
 		(at 72 52)
 		(size 0.6)
@@
 	)
 	(via
+		(at 178.9 76.4)
+		(size 0.6)
+		(drill 0.3)
+		(layers "F.Cu" "B.Cu")
+		(free yes)
+		(net 9)
+	)
+	(via
+		(at 178.9 93.4)
+		(size 0.6)
+		(drill 0.3)
+		(layers "F.Cu" "B.Cu")
+		(free yes)
+		(net 9)
+	)
+	(via
 		(at 197.75 117.8)
 		(size 0.6)
@@
 	)
 	(via
+		(at 206.4 77.4)
+		(size 0.6)
+		(drill 0.3)
+		(layers "F.Cu" "B.Cu")
+		(free yes)
+		(net 9)
+	)
+	(via
 		(at 123 117.824)
 		(size 0.6)
@@
 	)
 	(via
+		(at 168.2 60)
+		(size 0.6)
+		(drill 0.3)
+		(layers "F.Cu" "B.Cu")
+		(free yes)
+		(net 9)
+	)
+	(via
 		(at 129.7 48.9)
 		(size 0.6)
@@
 	)
 	(via
+		(at 183.3 101.4)
+		(size 0.6)
+		(drill 0.3)
+		(layers "F.Cu" "B.Cu")
+		(free yes)
+		(net 9)
+	)
+	(via
 		(at 114.5 38)
 		(size 0.6)
@@
 	)
 	(segment
-		(start 209.7 136.8)
-		(end 209.7 139.4)
-		(width 0.6)
-		(layer "B.Cu")
-		(net 9)
-	)
-	(segment
 		(start 209.7 100)
 		(end 209.7 117.9)
@@
 		(net 250)
 	)
+	(zone
+		(net 9)
+		(net_name "GND")
+		(layers "F.Cu" "B.Cu")
+		(hatch edge 0.5)
+		(connect_pads
+			(clearance 0.5)
+		)
+		(min_thickness 0.25)
+		(filled_areas_thickness no)
+		(fill yes
+			(thermal_gap 0.5)
+			(thermal_bridge_width 0.5)
+		)
+		(polygon
+			(pts
+				(xy 213 32) (xy 213 143.5) (xy 65 143.5) (xy 65 32)
+			)
+		)
+	)
 	(embedded_fonts no)
