File: Hardware/ECU/Inputs2.kicad_sch (KiCad schematic)
At the start: 10 parts, among them Q2 Q_DUAL_NMOS_S1G1D2S2G2D1, U14 LMV324LIDT

Commit message: PCB
Platine Vernetzt
Connections:
- net SPARE1-Digital renamed Tip Over Sensor
Other:
- note added: "Tip Over Sensor"
Changed lines of the file:
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@@
 	(text "Spare digital inputs"
 		(exclude_from_sim no)
-		(at 128.27 118.11 0)
+		(at 154.686 124.46 0)
 		(effects
 			(font
@@
 		(exclude_from_sim no)
 		(at 130.81 41.91 0)
+		(effects
+			(font
+				(size 1.8796 1.8796)
+			)
+			(justify left bottom)
+		)
+	)
+	(text "Tip Over Sensor"
+		(exclude_from_sim no)
+		(at 97.536 124.714 0)
 		(effects
 			(font
@@
 		)
 	)
-	(global_label "SPARE1-Digital"
+	(global_label "Tip Over Sensor"
 		(shape input)
 		(at 120.65 147.32 0)
@@
 		)
 		(property "Intersheetrefs" "${INTERSHEET_REFS}"
-			(at 137.8391 147.32 0)
+			(at 138.8751 147.32 0)
 			(effects
 				(font

Commit message: PCB v0.2
leiterbahndicke updated
Clutch input rework
Connections:
- net SPARE1_Sensor renamed Gear_Position
Changed lines of the file:
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@@
 		)
 	)
-	(global_label "SPARE1_Sensor"
+	(global_label "Gear_Position"
 		(shape input)
 		(at 105.41 49.53 180)
@@
 		)
 		(property "Intersheetrefs" "${INTERSHEET_REFS}"
-			(at 88.5838 49.53 0)
+			(at 89.483 49.53 0)
 			(effects
 				(font

Commit message: modified:   Hardware/ECU/Conntectors.kicad_sch deleted:    Hardware/ECU/ECU-backups/ECU-2025-05-14_000421.zip deleted:    Hardware/ECU/ECU-backups/ECU-2025-05-14_001426.zip deleted:    Hardware/ECU/ECU-backups/ECU-2025-05-14_002531.zip deleted:    Hardware/ECU/ECU-backups/ECU-2025-05-14_003555.zip deleted:    Hardware/ECU/ECU-backups/ECU-2025-05-14_004055.zip modified:   Hardware/ECU/ECU.kicad_pcb modified:   Hardware/ECU/ECU.kicad_prl modified:   Hardware/ECU/ECU.kicad_pro modified:   Hardware/ECU/ECU.kicad_sch 	modified:   Hardware/ECU/Inputs.kicad_sch 	modified:   Hardware/ECU/Inputs2.kicad_sch 	modified:   Hardware/ECU/Schematics.pdf 	modified:   Hardware/ECU/docs/Pinout.ods 	Hardware/ECU/ECU-backups/ECU-2025-05-19_135220.zip 	Hardware/ECU/ECU-backups/ECU-2025-05-19_140656.zip 	Hardware/ECU/ECU-backups/ECU-2025-05-19_142320.zip 	Hardware/ECU/ECU-backups/ECU-2025-05-19_145225.zip 	Hardware/ECU/ECU-backups/ECU-2025-05-19_160311.zip 	Hardware/ECU/ECU.kicad_pcb.zip 	Hardware/ECU/docs/GPS.JPG 	docs/Kabelplan.pdn
Parts:
- removed R48: 180k, Resistor_SMD:R_0805_2012Metric, symbol Device:R
- R49: value 348k -> 1k
Connections:
- net GND: no longer R49.1
- net Gear_Position: now also R49.2, U14.3 (+)
- new net +5V: R49.1
Changed lines of the file:
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@@
 	(wire
 		(pts
-			(xy 105.41 49.53) (xy 107.95 49.53)
+			(xy 105.41 49.53) (xy 118.11 49.53)
 		)
 		(stroke
@@
 		(pts
 			(xy 154.94 147.32) (xy 156.21 147.32)
-		)
-		(stroke
-			(width 0)
-			(type default)
-		)
-	)
-	(wire
-		(pts
-			(xy 118.11 49.53) (xy 115.57 49.53)
 		)
 		(stroke
@@
 	)
 	(symbol
+		(lib_id "power:+5V")
+		(at 129.54 49.53 270)
+		(unit 1)
+		(exclude_from_sim no)
+		(in_bom yes)
+		(on_board yes)
+		(dnp no)
+		(fields_autoplaced yes)
+		(property "Reference" "#PWR08"
+			(at 125.73 49.53 0)
+			(effects
+				(font
+					(size 1.27 1.27)
+				)
+				(hide yes)
+			)
+		)
+		(property "Value" "+5V"
+			(at 133.35 49.5299 90)
+			(effects
+				(font
+					(size 1.27 1.27)
+				)
+				(justify left)
+			)
+		)
+		(property "Footprint" ""
+			(at 129.54 49.53 0)
+			(effects
+				(font
+					(size 1.27 1.27)
+				)
+				(hide yes)
+			)
+		)
+		(property "Datasheet" ""
+			(at 129.54 49.53 0)
+			(effects
+				(font
+					(size 1.27 1.27)
+				)
+				(hide yes)
+			)
+		)
+		(property "Description" "Power symbol creates a global label with name \"+5V\""
+			(at 129.54 49.53 0)
+			(effects
+				(font
+					(size 1.27 1.27)
+				)
+				(hide yes)
+			)
+		)
+		(pin "1"
+		)
+		(instances
+			(project ""
+				(path "/aaebd8f9-fdac-426b-87c0-a208167b6035/208a416e-a5c2-4c6c-835c-57e49c0491be"
+					(reference "#PWR08")
+					(unit 1)
+				)
+			)
+		)
+	)
+	(symbol
 		(lib_id "power:GND")
 		(at 156.21 139.7 180)
@@
 			)
 		)
-		(property "Value" "348k"
+		(property "Value" "1k"
 			(at 124.46 46.5836 90)
 			(effects
@@
 	)
 	(symbol
-		(lib_id "Device:R")
-		(at 111.76 49.53 270)
-		(unit 1)
-		(exclude_from_sim no)
-		(in_bom yes)
-		(on_board yes)
-		(dnp no)
-		(property "Reference" "R48"
-			(at 111.76 44.2722 90)
-			(effects
-				(font
-					(size 1.27 1.27)
-				)
-			)
-		)
-		(property "Value" "180k"
-			(at 111.76 46.5836 90)
-			(effects
-				(font
-					(size 1.27 1.27)
-				)
-			)
-		)
-		(property "Footprint" "Resistor_SMD:R_0805_2012Metric"
-			(at 111.76 47.752 90)
-			(effects
-				(font
-					(size 1.27 1.27)
-				)
-				(hide yes)
-			)
-		)
-		(property "Datasheet" "~"
-			(at 111.76 49.53 0)
-			(effects
-				(font
-					(size 1.27 1.27)
-				)
-				(hide yes)
-			)
-		)
-		(property "Description" ""
-			(at 111.76 49.53 0)
-			(effects
-				(font
-					(size 1.27 1.27)
-				)
-				(hide yes)
-			)
-		)
-		(property "Digikey Part Number" "311-180KCRCT-ND"
-			(at 111.76 49.53 0)
-			(effects
-				(font
-					(size 1.27 1.27)
-				)
-				(hide yes)
-			)
-		)
-		(property "Manufacturer_Name" "Yageo"
-			(at 111.76 49.53 0)
-			(effects
-				(font
-					(size 1.27 1.27)
-				)
-				(hide yes)
-			)
-		)
-		(property "Manufacturer_Part_Number" "RC0805FR-07180KL"
-			(at 111.76 49.53 0)
-			(effects
-				(font
-					(size 1.27 1.27)
-				)
-				(hide yes)
-			)
-		)
-		(property "URL" "https://www.digikey.com.au/product-detail/en/yageo/RC0805FR-07180KL/311-180KCRCT-ND/730597"
-			(at 111.76 49.53 0)
-			(effects
-				(font
-					(size 1.27 1.27)
-				)
-				(hide yes)
-			)
-		)
-		(pin "1"
-		)
-		(pin "2"
-		)
-		(instances
-			(project "ECU"
-				(path "/aaebd8f9-fdac-426b-87c0-a208167b6035/208a416e-a5c2-4c6c-835c-57e49c0491be"
-					(reference "R48")
-					(unit 1)
-				)
-			)
-		)
-	)
-	(symbol
 		(lib_id "Amplifier_Operational:LMV324")
 		(at 166.37 59.69 270)
@@
 					(unit 1)
 				)
-			)
-		)
-	)
-	(symbol
-		(lib_id "power:GND")
-		(at 129.54 49.53 90)
-		(unit 1)
-		(exclude_from_sim no)
-		(in_bom yes)
-		(on_board yes)
-		(dnp no)
-		(property "Reference" "#PWR079"
-			(at 135.89 49.53 0)
-			(effects
-				(font
-					(size 1.27 1.27)
-				)
-				(hide yes)
-			)
-		)
-		(property "Value" "GND"
-			(at 132.7912 49.403 90)
-			(effects
-				(font
-					(size 1.27 1.27)
-				)
-				(justify right)
-			)
-		)
-		(property "Footprint" ""
-			(at 129.54 49.53 0)
-			(effects
-				(font
-					(size 1.27 1.27)
-				)
-				(hide yes)
-			)
-		)
-		(property "Datasheet" ""
-			(at 129.54 49.53 0)
-			(effects
-				(font
-					(size 1.27 1.27)
-				)
-				(hide yes)
-			)
-		)
-		(property "Description" ""
-			(at 129.54 49.53 0)
-			(effects
-				(font
-					(size 1.27 1.27)
-				)
-				(hide yes)
-			)
-		)
-		(pin "1"
-		)
-		(instances
-			(project "ECU"
-				(path "/aaebd8f9-fdac-426b-87c0-a208167b6035/208a416e-a5c2-4c6c-835c-57e49c0491be"
-					(reference "#PWR079")
-					(unit 1)
-				)

Commit message: deleted:    Hardware/ECU/ECU-backups/ECU-2025-05-27_235240.zip 	deleted:    Hardware/ECU/ECU-backups/ECU-2025-05-28_135321.zip 	deleted:    Hardware/ECU/ECU-backups/ECU-2025-05-28_140049.zip 	deleted:    Hardware/ECU/ECU-backups/ECU-2025-05-28_141416.zip 	deleted:    Hardware/ECU/ECU-backups/ECU-2025-05-28_154718.zip 	deleted:    Hardware/ECU/ECU-backups/ECU-2025-06-18_111329.zip 	new file:   Hardware/ECU/ECU-backups/ECU-2025-08-26_154141.zip 	new file:   Hardware/ECU/ECU-backups/ECU-2025-08-29_143817.zip 	new file:   Hardware/ECU/ECU-backups/ECU-2025-09-19_081818.zip 	new file:   Hardware/ECU/ECU-backups/ECU-2026-01-19_151411.zip 	new file:   Hardware/ECU/ECU-backups/ECU-2026-01-19_152057.zip 	new file:   Hardware/ECU/ECU-backups/ECU-2026-01-19_154705.zip 	modified:   Hardware/ECU/ECU.kicad_pcb 	modified:   Hardware/ECU/ECU.kicad_prl 	modified:   Hardware/ECU/ECU.kicad_sch 	modified:   Hardware/ECU/Inputs.kicad_sch 	modified:   Hardware/ECU/Inputs2.kicad_sch 	renamed:    Hardware/ECU/output/PCB.pdf -> Hardware/ECU/output/PCB-R9.3.pdf 	renamed:    Hardware/ECU/output/Schematics.pdf -> Hardware/ECU/output/Schematics-R0.3.pdf 	new file:   Hardware/ECU/output/Schematics-R1.pdf 	deleted:    Hardware/ECU/output/cut files/ECU-B_Cu.jpg 	modified:   speeduino (modified content)
Changed lines of the file:
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@@
 		)
 	)
-	(global_label "MCU-A17"
+	(global_label "MCU-A16"
 		(shape input)
 		(at 118.11 67.31 0)
@@
 		)
 		(property "Intersheetrefs" "${INTERSHEET_REFS}"
-			(at 129.4935 67.31 0)
+			(at 130.2271 67.31 0)
 			(effects
 				(font
@@
 		)
 	)
-	(global_label "MCU-A18"
+	(global_label "MCU-A17"
 		(shape input)
 		(at 168.91 67.31 0)
@@
 		)
 		(property "Intersheetrefs" "${INTERSHEET_REFS}"
-			(at 180.2935 67.31 0)
+			(at 181.0271 67.31 0)
 			(effects
 				(font
