File: hardware/ECU/Crank-and-Cam.kicad_sch (KiCad schematic)
At the start: 22 parts, among them IC1 MAX9926UAEE_V+, Q1 Q_DUAL_NMOS_S1G1D2S2G2D1, SW1 SW_DPDT_x2, SW2 SW_DPDT_x2

Commit message: Replace speeduino submodule with HasiKe fork, fix teensy.pretty path
- Switch speeduino from speeduino/speeduino to HasiKe/speeduino
- Fix teensy.pretty submodule path case mismatch (Hardware -> hardware)
- Add ISL9V5036P3-F085 component library
- Various ECU schematic updates
Parts:
- renumbered JP1 to JP4, R3 to R4, R4 to R5, R5 to R6, R6 to R7, R7 to R8, R8 to R9
Connections:
- net MCU-D18 renamed MCU-D21
- net MCU-D19 renamed MCU-D20
Changed lines of the file:
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@@
 		)
 	)
-	(global_label "MCU-D18"
+	(global_label "MCU-D21"
 		(shape input)
 		(at 128.27 99.06 0)
@@
 		)
 		(property "Intersheetrefs" "${INTERSHEET_REFS}"
-			(at 139.8349 99.06 0)
+			(at 140.5685 99.06 0)
 			(effects
 				(font
@@
 		)
 	)
-	(global_label "MCU-D19"
+	(global_label "MCU-D20"
 		(shape input)
 		(at 128.27 83.82 0)
@@
 		)
 		(property "Intersheetrefs" "${INTERSHEET_REFS}"
-			(at 139.8349 83.82 0)
+			(at 140.5685 83.82 0)
 			(effects
 				(font
@@
 		(on_board yes)
 		(dnp no)
-		(property "Reference" "#PWR022"
+		(property "Reference" "#PWR033"
 			(at 96.52 106.68 0)
 			(effects
@@
 			(project "ECU"
 				(path "/aaebd8f9-fdac-426b-87c0-a208167b6035/34d8184b-485a-4241-8a68-5c8e24cc7ad9"
-					(reference "#PWR022")
+					(reference "#PWR033")
 					(unit 1)
 				)
@@
 		(on_board yes)
 		(dnp no)
-		(property "Reference" "R5"
+		(property "Reference" "R6"
 			(at 246.38 76.2 90)
 			(effects
@@
 			(project "ECU"
 				(path "/aaebd8f9-fdac-426b-87c0-a208167b6035/34d8184b-485a-4241-8a68-5c8e24cc7ad9"
-					(reference "R5")
+					(reference "R6")
 					(unit 1)
 				)
@@
 		(on_board yes)
 		(dnp no)
-		(property "Reference" "R3"
+		(property "Reference" "R4"
 			(at 105.5878 80.01 90)
 			(effects
@@
 			(project "ECU"
 				(path "/aaebd8f9-fdac-426b-87c0-a208167b6035/34d8184b-485a-4241-8a68-5c8e24cc7ad9"
-					(reference "R3")
+					(reference "R4")
 					(unit 1)
 				)
@@
 		(on_board yes)
 		(dnp no)
-		(property "Reference" "#PWR024"
+		(property "Reference" "#PWR035"
 			(at 119.38 53.34 0)
 			(effects
@@
 			(project "ECU"
 				(path "/aaebd8f9-fdac-426b-87c0-a208167b6035/34d8184b-485a-4241-8a68-5c8e24cc7ad9"
-					(reference "#PWR024")
+					(reference "#PWR035")
 					(unit 1)
 				)
@@
 		(on_board yes)
 		(dnp no)
-		(property "Reference" "R6"
+		(property "Reference" "R7"
 			(at 246.38 83.82 90)
 			(effects
@@
 			(project "ECU"
 				(path "/aaebd8f9-fdac-426b-87c0-a208167b6035/34d8184b-485a-4241-8a68-5c8e24cc7ad9"
-					(reference "R6")
+					(reference "R7")
 					(unit 1)
 				)
@@
 		(on_board yes)
 		(dnp no)
-		(property "Reference" "R7"
+		(property "Reference" "R8"
 			(at 246.38 96.52 90)
 			(effects
@@
 			(project "ECU"
 				(path "/aaebd8f9-fdac-426b-87c0-a208167b6035/34d8184b-485a-4241-8a68-5c8e24cc7ad9"
-					(reference "R7")
+					(reference "R8")
 					(unit 1)
 				)
@@
 		(on_board yes)
 		(dnp no)
-		(property "Reference" "#PWR028"
+		(property "Reference" "#PWR039"
 			(at 248.92 93.98 0)
 			(effects
@@
 			(project "ECU"
 				(path "/aaebd8f9-fdac-426b-87c0-a208167b6035/34d8184b-485a-4241-8a68-5c8e24cc7ad9"
-					(reference "#PWR028")
+					(reference "#PWR039")
 					(unit 1)
 				)
@@
 		(on_board yes)
 		(dnp no)
-		(property "Reference" "#PWR027"
+		(property "Reference" "#PWR038"
 			(at 238.76 86.36 0)
 			(effects
@@
 			(project "ECU"
 				(path "/aaebd8f9-fdac-426b-87c0-a208167b6035/34d8184b-485a-4241-8a68-5c8e24cc7ad9"
-					(reference "#PWR027")
+					(reference "#PWR038")
 					(unit 1)
 				)
@@
 		(on_board yes)
 		(dnp no)
-		(property "Reference" "#PWR021"
+		(property "Reference" "#PWR032"
 			(at 96.52 76.2 0)
 			(effects
@@
 			(project "ECU"
 				(path "/aaebd8f9-fdac-426b-87c0-a208167b6035/34d8184b-485a-4241-8a68-5c8e24cc7ad9"
-					(reference "#PWR021")
+					(reference "#PWR032")
 					(unit 1)
 				)
@@
 		(on_board yes)
 		(dnp no)
-		(property "Reference" "#PWR026"
+		(property "Reference" "#PWR037"
 			(at 165.1 102.87 0)
 			(effects
@@
 			(project "ECU"
 				(path "/aaebd8f9-fdac-426b-87c0-a208167b6035/34d8184b-485a-4241-8a68-5c8e24cc7ad9"
-					(reference "#PWR026")
+					(reference "#PWR037")
 					(unit 1)
 				)
@@
 		(on_board yes)
 		(dnp no)
-		(property "Reference" "#PWR025"
+		(property "Reference" "#PWR036"
 			(at 165.1 77.47 0)
 			(effects
@@
 			(project "ECU"
 				(path "/aaebd8f9-fdac-426b-87c0-a208167b6035/34d8184b-485a-4241-8a68-5c8e24cc7ad9"
-					(reference "#PWR025")
+					(reference "#PWR036")
 					(unit 1)
 				)
@@
 		(on_board yes)
 		(dnp no)
-		(property "Reference" "R8"
+		(property "Reference" "R9"
 			(at 246.38 104.14 90)
 			(effects
@@
 			(project "ECU"
 				(path "/aaebd8f9-fdac-426b-87c0-a208167b6035/34d8184b-485a-4241-8a68-5c8e24cc7ad9"
-					(reference "R8")
+					(reference "R9")
 					(unit 1)
 				)
@@
 		(on_board yes)
 		(dnp no)
-		(property "Reference" "R4"
+		(property "Reference" "R5"
 			(at 105.41 102.87 90)
 			(effects
@@
 			(project "ECU"
 				(path "/aaebd8f9-fdac-426b-87c0-a208167b6035/34d8184b-485a-4241-8a68-5c8e24cc7ad9"
-					(reference "R4")
+					(reference "R5")
 					(unit 1)
 				)
@@
 		(on_board yes)
 		(dnp no)
-		(property "Reference" "#PWR023"
+		(property "Reference" "#PWR034"
 			(at 113.03 118.11 0)
 			(effects
@@
 			(project "ECU"
 				(path "/aaebd8f9-fdac-426b-87c0-a208167b6035/34d8184b-485a-4241-8a68-5c8e24cc7ad9"
-					(reference "#PWR023")
+					(reference "#PWR034")
 					(unit 1)
 				)
@@
 		(on_board yes)
 		(dnp no)
-		(property "Reference" "JP1"
+		(property "Reference" "JP4"
 			(at 112.141 76.2 0)
 			(effects
@@
 			(project "ECU"
 				(path "/aaebd8f9-fdac-426b-87c0-a208167b6035/34d8184b-485a-4241-8a68-5c8e24cc7ad9"
-					(reference "JP1")
+					(reference "JP4")
 					(unit 1)
 				)
