File: hardware/ECU/Crank-and-Cam.kicad_sch (KiCad schematic)
At the start: 22 parts, among them IC1 MAX9926UAEE_V+, Q1 Q_DUAL_NMOS_S1G1D2S2G2D1, SW1 SW_DPDT_x2, SW2 SW_DPDT_x2

Commit message: Update ECU-Hardware, Dokumente und Explosionszeichnungen
Parts:
- removed C3: 0.1uF, Capacitor_SMD:C_0805_2012Metric, symbol Device:C
- removed C4: 0.01uF, Capacitor_SMD:C_0805_2012Metric, symbol Device:C
- removed C5: 4700pF, Capacitor_SMD:C_0805_2012Metric, symbol Device:C
- removed JP2, JP3, JP4, JP5: Jumper_2_Open, Jumper:SolderJumper-2_P1.3mm_Open_Pad1.0x1.5mm, symbol Jumper:Jumper_2_Open
- removed Q1: Q_DUAL_NMOS_S1G1D2S2G2D1, Package_TO_SOT_SMD:SOT-363_SC-70-6, symbol Device:Q_DUAL_NMOS_S1G1D2S2G2D1
- removed R4, R5: 1k, Resistor_SMD:R_0805_2012Metric, symbol Device:R
- removed SW1, SW2: SW_DPDT_x2, Misc:AYZ0202AGRLC, symbol Switch:SW_SPDT
- added C8, C9: 470pF, Capacitor_SMD:C_0805_2012Metric, symbol Device:C
- added D4, D5, D6, D7: BAV199, Package_TO_SOT_SMD:SOT-23, symbol Diode:BAV199
- added R10, R21, R22, R9: 0R DNP, Resistor_SMD:R_0805_2012Metric, symbol Device:R
- added R11, R13, R19, R20: 0R, Resistor_SMD:R_0805_2012Metric, symbol Device:R
- added R12, R14: 470R, Resistor_SMD:R_0805_2012Metric, symbol Device:R
- added R15, R16: 10k DNP, Resistor_SMD:R_0805_2012Metric, symbol Device:R
- added R17, R18: 1k, Resistor_SMD:R_0805_2012Metric, symbol Device:R
- C10: renamed from C6; Supplier (none) -> DigiKey
- C11: renamed from C7; Supplier (none) -> DigiKey
- C12: renamed from C8; Supplier (none) -> DigiKey
- C13: renamed from C9; Supplier (none) -> DigiKey
- C14: renamed from C10; Supplier (none) -> DigiKey
- IC1: Manufacturer_Name Maxim Integrated -> Analog Devices; Supplier (none) -> DigiKey
- R23: renamed from R6; Supplier (none) -> DigiKey
- R24: renamed from R7; Supplier (none) -> DigiKey
- R25: renamed from R8; Supplier (none) -> DigiKey
- R26: renamed from R9; Supplier (none) -> DigiKey
Connections:
- net +3V3: now also D4.2 (K2), D5.2 (K2), D6.2 (K2), D7.2 (K2), R15.2, R16.2
- net CAM-IN+: now also R10.1, R13.1
- net CRANK-IN+: now also R11.1, R9.1
- net GND: now also C8.2, C9.2, D4.1 (A1), D5.1 (A1), D6.1 (A1), D7.1 (A1)
- net MCU-D20: now also C8.1, D4.3 (K1A2), R12.2; no longer IC1.4 (COUT1)
- net MCU-D21: now also C9.1, D5.3 (K1A2), R14.2; no longer IC1.5 (COUT2)
- net VR1-IN+: now also R11.2
- net VR2-IN+: now also R13.2
- new net: R10.2, R18.1
- new net: R17.1, R9.2
- new net CAM-HALL: D7.3 (K1A2), R16.1, R18.2, R22.1
- new net CAM-SIG: R14.1, R20.2, R22.2
- new net CRANK-HALL: D6.3 (K1A2), R15.1, R17.2, R21.1
- new net CRANK-SIG: R12.1, R19.2, R21.2
- new net VR1-OUT: IC1.4 (COUT1), R19.1
- new net VR2-OUT: IC1.5 (COUT2), R20.1
Other:
- note added: "CAM: VR-Pfad (0R bestueckt) oder Hall-Pfad (0R DNP) - Rev 3.0 ohne Schiebeschalter"
- note added: "CRANK: VR-Pfad (0R bestueckt) oder Hall-Pfad (0R DNP) - Rev 3.0 ohne Schiebeschalter"
- note added: "MAX9926 COUT = 5V Push-Pull -> 470R Serie + BAV199-Klemme an +3V3 am Teensy-Pin, 470pF Filter"
- note removed: "Circuit Reference: Phillips AN97055"
- note removed: "See VR Conditioner"
- title: (none) -> Crank and Cam
- moved on the sheet: C13, C14
