File: hardware/ECU/Outputs.kicad_sch (KiCad schematic)
At the start: 25 parts, among them IC2 ZXMS6006DT8, IC3 ZXMS6006DT8, IC4 ZXMS6006DT8

Commit message: Replace speeduino submodule with HasiKe fork, fix teensy.pretty path
- Switch speeduino from speeduino/speeduino to HasiKe/speeduino
- Fix teensy.pretty submodule path case mismatch (Hardware -> hardware)
- Add ISL9V5036P3-F085 component library
- Various ECU schematic updates
Parts:
- added D18: LED, LED_SMD:LED_0805_2012Metric, symbol Device:LED
- added D19: D, Diode_SMD:D_SOD-323, symbol Device:D
- added IC3: ZXMS6006DT8, ZXMS6006DT8TA:SOT153P700X170-8N, symbol IC_Automotive:ZXMS6006DT8
- added R51, R52: 1k, Resistor_SMD:R_0805_2012Metric, symbol Device:R
- added R55, R56: 100k, Resistor_SMD:R_0805_2012Metric, symbol Device:R
- added R58: 10k, Resistor_SMD:R_0805_2012Metric, symbol Device:R
- R57: value 10k -> 1k; Digikey Part Number 311-10KARCT-ND -> 311-1.00KCRCT-ND; Manufacturer_Part_Number RC0805JR-0710KL -> RC0805FR-071KL; URL https://www.digikey.com/product-detail/en/yageo/RC0805JR-07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 -> https://www.digikey.com/product-detail/en/yageo/RC0805FR-07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
- renumbered C31 to C30, D25 to D15, D26 to D16, D27 to D17, D28 to D20, D29 to D21, D30 to D22, D31 to D23, IC3 to IC4, IC4 to IC5, R53 to R49, R54 to R50, R55 to R53, R56 to R54, R58 to R59, R59 to R60, R60 to R61, R61 to R62, R62 to R63, R63 to R64, R64 to R65, R65 to R66
Connections:
- net ROUT2 is gone; now on net 12V-SW: R57.1
- net 12V-SW: now also D19.1 (K), R58.2; no longer R57.2
- net FUELPUMP-OUT: now also D18.1 (K), D19.2 (A), IC3.7 (DRAIN_1_1), IC3.8 (DRAIN_1_2)
- net GND: now also IC3.2 (SOURCE_1), IC3.4 (SOURCE_2), R55.2, R56.1
- new net: IC3.1 (INPUT_1), R51.1, R55.1
- new net: D18.2 (A), R57.2
- new net: IC3.3 (INPUT_2), R52.1, R56.2
- new net MCU-D5: R51.2
- new net MCU-D8: R52.2
- new net TACHO-OUT: IC3.5 (DRAIN_2_1), IC3.6 (DRAIN_2_2), R58.1
Other:
- note added: "Tacho and Fuel Pump relay"
- note removed: "Fuel pump relay"
- note removed: "Tacho output"
