File: hardware/ECU/Outputs.kicad_sch (KiCad schematic)
At the start: 33 parts, among them IC2 ZXMS6006DT8, IC3 ZXMS6006DT8, IC4 ZXMS6006DT8, IC5 ZXMS6006DT8

Commit message: Update ECU-Hardware, Dokumente und Explosionszeichnungen
Parts:
- removed A1: Pololu_Breakout_DRV8825, Module:Pololu_Breakout-16_15.2x20.3mm, symbol Driver_Motor:Pololu_Breakout_DRV8825
- removed C30: 100uF, Capacitor_SMD:CP_Elec_6.3x7.7, symbol Device:CP
- removed D15, D16, D19, D20, D21, D22, D23: D, Diode_SMD:D_SOD-323, symbol Device:D
- removed D17: D_Schottky, Diode_SMD:D_PowerDI-123, symbol Device:D_Schottky
- removed D18: LED, LED_SMD:LED_0805_2012Metric, symbol Device:LED
- removed IC5: ZXMS6006DT8, ZXMS6006DT8TA:SOT153P700X170-8N, symbol IC_Automotive:ZXMS6006DT8
- removed R49, R50, R59, R60, R61, R62: 1k, Resistor_SMD:R_0805_2012Metric_Pad1.20x1.40mm_HandSolder, symbol Device:R
- removed R51, R52, R57: 1k, Resistor_SMD:R_0805_2012Metric, symbol Device:R
- removed R53, R54, R63, R64, R65, R66: 100k, Resistor_SMD:R_0805_2012Metric_Pad1.20x1.40mm_HandSolder, symbol Device:R
- removed R55, R56: 100k, Resistor_SMD:R_0805_2012Metric, symbol Device:R
- removed R58: 10k, Resistor_SMD:R_0805_2012Metric, symbol Device:R
- added C44, C45: 10n, Capacitor_SMD:C_0805_2012Metric, symbol Device:C
- added C46: 100u/50V, Capacitor_SMD:CP_Elec_8x10, symbol Device:CP
- added C47: 1u, Capacitor_SMD:C_0805_2012Metric, symbol Device:C
- added C48: 220n, Capacitor_SMD:C_0805_2012Metric, symbol Device:C
- added C49: 22n, Capacitor_SMD:C_0805_2012Metric, symbol Device:C
- added C50: 1n, Capacitor_SMD:C_0805_2012Metric, symbol Device:C
- added C51, C52: 100n, Capacitor_SMD:C_0805_2012Metric, symbol Device:C
- added D31, D32, D33, D34, D35, D36, D39, D40: SS34, Diode_SMD:D_SMA, symbol Device:D_Schottky
- added D37, D38: 1N4148W, Diode_SMD:D_SOD-123, symbol Diode:1N4148WT
- added Q5: BSS138, Package_TO_SOT_SMD:SOT-23, symbol Device:Q_NMOS_GDS
- added R100, R101, R102, R103, R104, R108, R109, R112, R99: 100k, Resistor_SMD:R_0805_2012Metric, symbol Device:R
- added R105: 15k, Resistor_SMD:R_0805_2012Metric, symbol Device:R
- added R106, R110, R111, R113: 10k, Resistor_SMD:R_0805_2012Metric, symbol Device:R
- added R107: 330k, Resistor_SMD:R_0805_2012Metric, symbol Device:R
- added R93, R94, R95, R96, R97, R98: 1k, Resistor_SMD:R_0805_2012Metric, symbol Device:R
- added U12: DRV8434A, Package_SO:HTSSOP-28-1EP_4.4x9.7mm_P0.65mm_EP2.85x5.4mm_ThermalVias, symbol Rev3:DRV8434A
- added U13, U14: BTF3050TE, Package_TO_SOT_SMD:TO-252-5_TabPin3, symbol Rev3:BTF3050TE
- IC2, IC3, IC4: BOM Comments (none) -> Last Time Buy 06.01.2027 - Bedarf sichern; Height 1.75 -> (none); Manufacturer_Name Diodes Inc -> Diodes Incorporated; Manufacturer_Part_Number ZXMS6006DT8 -> ZXMS6006DT8TA; Supplier (none) -> DigiKey; URL https://www.digikey.com.au/en/products/detail/diodes-incorp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 -> (none)
Connections:
- net SPARE1-OUT is gone; now on net FAN-OUT: IC4.7 (DRAIN_1_1), IC4.8 (DRAIN_1_2)
- net +3V3: now also C51.1, C52.1, R113.1, U12.18 (M0), U12.22 (M1), U13.2 (VDD), U14.2 (VDD)
- net BOOST-OUT: now also D39.2 (A), U13.3 (OUT)
- net FAN-OUT: now also D35.2 (A)
- net FUELPUMP-OUT: now also D33.2 (A)
- net GND: now also C47.2, C50.2, C51.2, C52.2, Q5.3 (S), R100.2, R101.2, R102.2, R103.2, R104.2, R106.2, R107.2, R108.1, R109.1, R110.2, R111.2, R112.2, R99.2, U12.14 (GND), U12.29 (PAD); no longer IC2.2 (SOURCE_1), IC2.4 (SOURCE_2), IC3.2 (SOURCE_1), IC3.4 (SOURCE_2), IC4.2 (SOURCE_1), IC4.4 (SOURCE_2)
- net MCU-D24: now also R108.2, U13.1 (IN)
- net MCU-D25: now also R109.2, U14.1 (IN)
- net MCU-D26: now also R94.1
- net MCU-D27: now also R93.1
- net MCU-D28: now also R98.1
- net MCU-D29: now also R97.1
- net MCU-D30: now also U12.23 (STEP)
- net MCU-D31: now also U12.24 (DIR)
- net MCU-D32: now also U12.25 (ENABLE), U12.26 (nSLEEP)
- net MCU-D5: now also R95.1
- net MCU-D8: now also R96.1
- net STEPPER-A1: now also U12.4 (AOUT1), U12.5 (AOUT1)
- net STEPPER-A2: now also U12.6 (AOUT2), U12.7 (AOUT2)
- net STEPPER-B1: now also U12.10 (BOUT1), U12.11 (BOUT1)
- net STEPPER-B2: now also U12.8 (BOUT2), U12.9 (BOUT2)
- net TACHO-OUT: now also D34.2 (A)
- net G_FAN: now reaches IC4.1 (INPUT_1)
- net G_FAN: now also R103.1, R97.2
- net G_STRT: now reaches IC2.3 (INPUT_2)
- net G_STRT: now also R100.1, R94.2
- net G_FUEL: now reaches IC3.1 (INPUT_1)
- net G_FUEL: now also R101.1, R95.2
- net G_SPARE: now reaches IC4.3 (INPUT_2)
- net G_SPARE: now also R104.1, R98.2
- net G_FI: now reaches IC2.1 (INPUT_1)
- net G_FI: now also R93.2, R99.1
- net G_TACH: now reaches IC3.3 (INPUT_2)
- net G_TACH: now also R102.1, R96.2
- net IDLE-OUT renamed FI-LAMP
- net FI-LAMP: now also D31.2 (A)
- net SPARE2-OUT renamed STARTER-OUT
- net STARTER-OUT: now also D32.2 (A)
- net SPARE2_OUT renamed SPARE-OUT
- net SPARE-OUT: now also D36.2 (A)
- new net: C48.2, U12.1 (VCP)
- new net: C49.1, U12.27 (CPL)
- new net: C49.2, U12.28 (CPH)
- new net 12V-PROT: C44.1, C45.1, C46.1, C48.1, D31.1 (K), D32.1 (K), D33.1 (K), D34.1 (K), D35.1 (K), D36.1 (K), D39.1 (K), D40.1 (K), U12.13 (VM), U12.2 (VM)
- new net DRV_DVDD: C47.1, R105.1, U12.15 (DVDD)
- new net DRV_STLM: R107.1, U12.21 (STL_MODE)
- new net DRV_TRQ: C50.1, U12.20 (TRQ_CNT/STL_TH)
- new net DRV_VREF: R105.2, R106.1, U12.17 (VREF)
- new net MCU-D9: Q5.2 (D), R113.2, U12.16 (nFAULT)
- new net O2-HEATER: D40.2 (A), U14.3 (OUT)
- new net OUT-FAULT-H: D37.1 (K), D38.1 (K), Q5.1 (G), R112.1
- new net PGND: C44.2, C45.2, C46.2, IC2.2 (SOURCE_1), IC2.4 (SOURCE_2), IC3.2 (SOURCE_1), IC3.4 (SOURCE_2), IC4.2 (SOURCE_1), IC4.4 (SOURCE_2), U12.12 (PGND), U12.3 (PGND), U13.5 (GND), U14.5 (GND)
- new net SRP_BOOST: D37.2 (A), R110.1, U13.4 (SRP)
- new net SRP_O2: D38.2 (A), R111.1, U14.4 (SRP)
- no-connect marks 0 -> 1
Other:
- note added: "A) Gate-Netzwerke: MCU-Pin → 1k → Gate, 100k Pulldown (Boot-sicher aus)"
- note added: "B) ZXMS6006DT8 Dual-Low-Side — IC2: FI-Lampe / Starter-Relais, IC3: Kraftstoffpumpe / Tacho, IC4: Lüfter / Spare"
- note added: "C) BTF3050TE Smart-Low-Side (VDD=+3V3 → Status 3V3-sicher; R_SRP 10k = Slew/Status; Freilauf SS34 nach 12V-PROT)"
- note added: "D) Status-ODER: SRP high (Übertemperatur-Latch) → Diode → OUT-FAULT-H → BSS138 zieht MCU-D9 (nFAULT, wired-OR) auf low"
- note added: "DRV8434A Peripherie"
- note added: "E) DRV8434A Stepper (VM=12V-PROT, 1/8-Schritt, IFS = VREF/1.32 V/A = 1.0 A @ VREF 1.32 V, Stall-Erkennung aus, nFAULT → MCU-D9)"
- note removed: "Fan and Boost outputs"
- note removed: "PWM Idle and Spare 2 outputs"
- note removed: "Stepper Driver (DRV8825)"
- note removed: "Tacho and Fuel Pump relay"
- note removed: "VVT and Spare 1"
- title: (none) -> Outputs
