File: hardware/ECU/Comms.kicad_sch (KiCad schematic)
At the start: 10 parts, among them J1 Conn_01x04, U2 W25Q32JVSS, U3 MCP2562-E-SN, U4 74AHC1G32, U5 ADXL343

Commit message: Update ECU-Hardware, Dokumente und Explosionszeichnungen
Parts:
- removed JP1: Jumper_NO_Small, Jumper:SolderJumper-2_P1.3mm_Open_Pad1.0x1.5mm, symbol Device:Jumper_NO_Small
- removed R3: 120R, Resistor_SMD:R_0805_2012Metric, symbol Device:R
- added C4: 4.7nF, Capacitor_SMD:C_0805_2012Metric, symbol Device:C
- added R2, R4, R5, R8: 10k, Resistor_SMD:R_0805_2012Metric, symbol Device:R
- added R6, R7: 60.4R, Resistor_SMD:R_0805_2012Metric, symbol Device:R
- C2: renamed from C1; Supplier (none) -> DigiKey
- C3: renamed from C2; Supplier (none) -> DigiKey
- J1: Digikey Part Number (none) -> 732-5317-ND; Manufacturer_Name (none) -> Würth Elektronik; Manufacturer_Part_Number (none) -> 61300411121; Supplier (none) -> DigiKey
- R3: renamed from R2; value 0R -> 10k; Digikey Part Number 311-0.0ARCT-ND -> 311-10.0KCRCT-ND; Manufacturer_Part_Number RC0805JR-070RL -> RC0805FR-0710KL; Supplier (none) -> DigiKey
- U2: BOM Comments (none) -> Nur ~39 St. bei DigiKey; Alternative W25Q32JVSSIQ via Mouser; Digikey Part Number W25Q32JVSSIQCT-ND -> 256-W25Q32RVCSJQTR-ND; Manufacturer_Name Winbond Electronics -> Winbond; Manufacturer_Part_Number W25Q32JVSSIQ -> W25Q32RVCSJQ TR; Supplier (none) -> DigiKey
- U3, U5: Supplier (none) -> DigiKey
- U4: Manufacturer_Name Analog Devices -> Texas Instruments; Supplier (none) -> DigiKey
Connections:
- net +3V3: now also R2.1, R4.1, R5.1, R8.1; no longer U2.3 (IO2), U2.7 (IO3)
- net CAN_H: now also R6.1
- net CAN_L: now also R7.2
- net GND: now also C4.2
- net MCU-D6: now also R2.2
- net MCU-D7: now also R8.2
- net VDD renamed +5V
- new net: C4.1, R6.2, R7.1
- new net: R5.2, U2.7 (IO3)
- new net: R4.2, U2.3 (IO2)
Other:
- title: (none) -> Communication
