File: hardware/ECU/ECU.kicad_pcb (KiCad board)
At the start: 2 copper layers, 148 x 111.5 mm, 172 parts, among them IC1 MAX9926UAEE_V+, IC2 ZXMS6006DT8, IC3 ZXMS6006DT8, IC4 ZXMS6006DT8, IC5 ZXMS6006DT8, J1 Conn_01x04, Q1 Q_DUAL_NMOS_S1G1D2S2G2D1, Q2 ISL9V5036P3-F085, Q3 ISL9V5036P3-F085, Q4 ISL9V5036P3-F085, Q5 ISL9V5036P3-F085, Q6 Q_DUAL_NMOS_S1G1D2S2G2D1, SW1 SW_DPDT_x2, SW2 SW_DPDT_x2, SW3 SW_DPDT_x2, U1 Teensy4.1, U10 SP720, U11 LMV324LIDT, U12 MC78M05_TO252, U2 W25Q32JVSS, U3 MCP2562-E-SN, U4 74AHC1G32, U5 ADXL343, U6 TC4424A, U7 MC33810, U8 TC4424A, U9 LMV324LIDT

Commit message: Update ECU-Hardware, Dokumente und Explosionszeichnungen
Parts:
- removed A1: Pololu_Breakout_DRV8825, Module:Pololu_Breakout-16_15.2x20.3mm
- removed JP1: Jumper_NO_Small, Jumper:SolderJumper-2_P1.3mm_Open_Pad1.0x1.5mm
- removed JP2, JP3, JP4, JP5, JP6: Jumper_2_Open, Jumper:SolderJumper-2_P1.3mm_Open_Pad1.0x1.5mm
- removed SW1, SW2, SW3: SW_DPDT_x2, Misc:AYZ0202AGRLC
- added C38: 100nF, Capacitor_SMD:C_0805_2012Metric, F.Cu at (114.0, 116.0)
- added C39: 10nF, Capacitor_SMD:C_0805_2012Metric, F.Cu at (118.0, 115.0)
- added C40: 10nF, Capacitor_SMD:C_0805_2012Metric, F.Cu at (126.0, 116.0)
- added C41: 100nF, Capacitor_SMD:C_0805_2012Metric, F.Cu at (127.5, 97.0)
- added C42: 100nF, Capacitor_SMD:C_0805_2012Metric, F.Cu at (114.0, 100.5)
- added C43: 100nF, Capacitor_SMD:C_0805_2012Metric, F.Cu at (127.0, 132.0)
- added C44: 10n, Capacitor_SMD:C_0805_2012Metric, F.Cu at (203.5, 100.0)
- added C45: 10n, Capacitor_SMD:C_0805_2012Metric, F.Cu at (161.0, 98.5)
- added C46: 100u/50V, Capacitor_SMD:CP_Elec_8x10, F.Cu at (195.0, 106.5)
- added C47: 1u, Capacitor_SMD:C_0805_2012Metric, F.Cu at (127.0, 34.8)
- added C48: 220n, Capacitor_SMD:C_0805_2012Metric, F.Cu at (116.6, 34.8)
- added C49: 22n, Capacitor_SMD:C_0805_2012Metric, F.Cu at (124.4, 34.8)
- added C50: 1n, Capacitor_SMD:C_0805_2012Metric, F.Cu at (129.6, 34.8)
- added C51: 100n, Capacitor_SMD:C_0805_2012Metric, F.Cu at (165.0, 99.0)
- added C52: 100n, Capacitor_SMD:C_0805_2012Metric, F.Cu at (165.5, 95.0)
- added C53: 100nF/100V, Capacitor_SMD:C_1210_3225Metric, F.Cu at (111.5, 131.5)
- added C54: 100nF/100V, Capacitor_SMD:C_1210_3225Metric, F.Cu at (105.0, 140.0)
- added C55: 4.7uF/100V, Capacitor_SMD:C_1210_3225Metric, F.Cu at (117.5, 129.5)
- added C56: 4.7uF/100V, Capacitor_SMD:C_1210_3225Metric, F.Cu at (111.5, 127.0)
- added C57: 1uF/50V, Capacitor_SMD:C_0805_2012Metric, F.Cu at (76.5, 139.5)
- added C58: 10uF/10V, Capacitor_SMD:C_0805_2012Metric, F.Cu at (119.0, 138.0)
- added C59: 100nF/25V, Capacitor_SMD:C_0805_2012Metric, F.Cu at (71.0, 115.5)
- added C60: 39pF, Capacitor_SMD:C_0805_2012Metric, F.Cu at (83.5, 133.0)
- added C61: 100uF/50V, Capacitor_SMD:CP_Elec_8x10, F.Cu at (87.5, 117.5)
- added C62: 6800pF, Capacitor_SMD:C_0805_2012Metric, F.Cu at (68.5, 115.5)
- added C63: 10uF/10V, Capacitor_SMD:C_0805_2012Metric, F.Cu at (109.0, 80.5)
- added C64: 22uF/10V, Capacitor_SMD:C_1210_3225Metric, F.Cu at (113.0, 136.0)
- added C65: 100nF/100V, Capacitor_SMD:C_1210_3225Metric, F.Cu at (99.0, 140.0)
- added C66: 100nF/25V, Capacitor_SMD:C_0805_2012Metric, F.Cu at (73.0, 130.5)
- added C67: 100nF, Capacitor_SMD:C_0805_2012Metric, F.Cu at (124.5, 135.5)
- added C68: 100nF, Capacitor_SMD:C_0805_2012Metric, F.Cu at (114.0, 140.0)
- added C69: 100uF/50V, Capacitor_SMD:CP_Elec_8x10, F.Cu at (102.0, 132.5)
- added C70: 47uF/10V X7R, Capacitor_SMD:C_1210_3225Metric, F.Cu at (123.5, 128.0)
- added C71: 10uF/50V X7R, Capacitor_SMD:C_1210_3225Metric, F.Cu at (111.5, 122.5)
- added C72: 47uF/10V X7R, Capacitor_SMD:C_1210_3225Metric, F.Cu at (119.0, 134.0)
- added C73: 100nF/100V, Capacitor_SMD:C_1210_3225Metric, F.Cu at (117.5, 125.0)
- added C74: 100nF, Capacitor_SMD:C_0805_2012Metric, F.Cu at (69.0, 95.0)
- added C75: 0.01uF, Capacitor_SMD:C_0805_2012Metric, F.Cu at (153.0, 133.0)
- added C76: CC0805KRX7R9BB104, Capacitor_SMD:C_0805_2012Metric, F.Cu at (161.5, 94.5)
- added C77: 100nF, Capacitor_SMD:C_0805_2012Metric, F.Cu at (150.5, 92.5)
- added C78: CC0805KRX7R9BB104, Capacitor_SMD:C_0805_2012Metric, F.Cu at (162.5, 91.0)
- added C79: CC0805KKX7R7BB475, Capacitor_SMD:C_0805_2012Metric, F.Cu at (162.0, 87.5)
- added C80: CC0805KRX7R9BB104, Capacitor_SMD:C_0805_2012Metric, F.Cu at (158.0, 133.0)
- added C81: CC0805JRX7R9BB332, Capacitor_SMD:C_0805_2012Metric, F.Cu at (163.5, 139.0)
- added C82: CC0805JRX7R9BB332, Capacitor_SMD:C_0805_2012Metric, F.Cu at (154.5, 140.5)
- added D29: BAV199, Package_TO_SOT_SMD:SOT-23, F.Cu at (118.0, 120.0)
- added D30: BAV199, Package_TO_SOT_SMD:SOT-23, F.Cu at (114.5, 110.5)
- added D31: SS34, Diode_SMD:D_SMA, F.Cu at (192.5, 130.5)
- added D32: SS34, Diode_SMD:D_SMA, F.Cu at (185.5, 132.0)
- added D33: SS34, Diode_SMD:D_SMA, F.Cu at (196.0, 116.0)
- added D34: SS34, Diode_SMD:D_SMA, F.Cu at (198.5, 123.0)
- added D35: SS34, Diode_SMD:D_SMA, F.Cu at (179.0, 130.5)
- added D36: SS34, Diode_SMD:D_SMA, F.Cu at (179.0, 135.5)
- added D37: 1N4148W, Diode_SMD:D_SOD-123, F.Cu at (200.5, 117.0)
- added D38: 1N4148W, Diode_SMD:D_SOD-123, F.Cu at (170.0, 139.0)
- added D39: SS34, Diode_SMD:D_SMA, F.Cu at (206.5, 116.5)
- added D40: SS34, Diode_SMD:D_SMA, F.Cu at (176.0, 140.5)
- added D41: SM8S24A, Rev3:D_DO-218AB, F.Cu at (101.0, 102.0)
- added D42: B560C, Diode_SMD:D_SMC, F.Cu at (87.5, 126.5)
- added D43: LED grn, LED_SMD:LED_0805_2012Metric, F.Cu at (72.0, 85.5)
- added D44: LED grn, LED_SMD:LED_0805_2012Metric, F.Cu at (124.5, 139.0)
- added D45: LED grn, LED_SMD:LED_0805_2012Metric, F.Cu at (76.0, 81.5)
- added D46: BAV199, Package_TO_SOT_SMD:SOT-23, F.Cu at (163.0, 129.5)
- added D47: BAV199, Package_TO_SOT_SMD:SOT-23, F.Cu at (163.5, 134.5)
- added H1: M3, MountingHole:MountingHole_3.2mm_M3, F.Cu at (70.0, 138.5)
- added H2: M3, MountingHole:MountingHole_3.2mm_M3, F.Cu at (208.0, 138.5)
- added H3: M3, MountingHole:MountingHole_3.2mm_M3, F.Cu at (70.0, 37.0)
- added IC6: 74AHCT125T14-13, Package_SO:TSSOP-14_4.4x5mm_P0.65mm, F.Cu at (155.5, 119.5)
- added IC7: TPIC8101DW, Package_SO:SOIC-20W_7.5x12.8mm_P1.27mm, F.Cu at (158.0, 108.5)
- added L1: 10uH / 3.3A, Inductor_SMD:L_Bourns_SRR1260, F.Cu at (74.5, 104.5)
- added L2: 8.2uH / 5A, Inductor_SMD:L_Bourns_SRR1260, F.Cu at (100.5, 120.0)
- added NT1: NetTie_2, NetTie:NetTie-2_SMD_Pad0.5mm, F.Cu at (172.5, 76.0)
- added NT2: NetTie_2, NetTie:NetTie-2_SMD_Pad0.5mm, F.Cu at (169.5, 75.0)
- added R100: 100k, Resistor_SMD:R_0805_2012Metric, F.Cu at (203.0, 128.0)
- added R101: 100k, Resistor_SMD:R_0805_2012Metric, F.Cu at (199.0, 131.0)
- added R102: 100k, Resistor_SMD:R_0805_2012Metric, F.Cu at (190.5, 134.5)
- added R103: 100k, Resistor_SMD:R_0805_2012Metric, F.Cu at (209.0, 121.5)
- added R104: 100k, Resistor_SMD:R_0805_2012Metric, F.Cu at (196.5, 134.5)
- added R105: 15k, Resistor_SMD:R_0805_2012Metric, F.Cu at (119.2, 49.7)
- added R106: 10k, Resistor_SMD:R_0805_2012Metric, F.Cu at (119.2, 34.8)
- added R107: 330k, Resistor_SMD:R_0805_2012Metric, F.Cu at (121.8, 34.8)
- added R108: 100k, Resistor_SMD:R_0805_2012Metric, F.Cu at (185.5, 138.0)
- added R109: 100k, Resistor_SMD:R_0805_2012Metric, F.Cu at (189.5, 138.5)
- added R110: 10k, Resistor_SMD:R_0805_2012Metric, F.Cu at (207.0, 127.5)
- added R111: 10k, Resistor_SMD:R_0805_2012Metric, F.Cu at (204.5, 132.0)
- added R112: 100k, Resistor_SMD:R_0805_2012Metric, F.Cu at (200.0, 139.0)
- added R113: 10k, Resistor_SMD:R_0805_2012Metric, F.Cu at (116.6, 49.7)
- added R114: 237k, Resistor_SMD:R_0805_2012Metric, F.Cu at (80.5, 139.0)
- added R115: 56k2, Resistor_SMD:R_0805_2012Metric, F.Cu at (69.5, 131.0)
- added R116: 162k, Resistor_SMD:R_0805_2012Metric, F.Cu at (85.0, 138.0)
- added R117: 53k6, Resistor_SMD:R_0805_2012Metric, F.Cu at (72.5, 126.5)
- added R118: 10k2, Resistor_SMD:R_0805_2012Metric, F.Cu at (79.5, 135.5)
- added R119: 13k, Resistor_SMD:R_0805_2012Metric, F.Cu at (70.5, 122.5)
- added R120: 470R, Resistor_SMD:R_0805_2012Metric, F.Cu at (80.5, 72.0)
- added R121: 2k2, Resistor_SMD:R_0805_2012Metric, F.Cu at (128.0, 124.0)
- added R122: 1k, Resistor_SMD:R_0805_2012Metric, F.Cu at (78.5, 76.5)
- added R123: 10k, Resistor_SMD:R_0805_2012Metric, F.Cu at (158.0, 136.5)
- added R124: 1k, Resistor_SMD:R_0805_2012Metric, F.Cu at (153.0, 129.5)
- added R125: 2k, Resistor_SMD:R_0805_2012Metric, F.Cu at (153.0, 136.5)
- added R126: RC0805FR-071ML, Resistor_SMD:R_0805_2012Metric, F.Cu at (158.0, 129.5)
- added R127: RC0805FR-07100KL, Resistor_SMD:R_0805_2012Metric, F.Cu at (163.5, 122.0)
- added R128: RC0805FR-07100KL, Resistor_SMD:R_0805_2012Metric, F.Cu at (163.5, 125.5)
- added R129: RC0805FR-07100KL, Resistor_SMD:R_0805_2012Metric, F.Cu at (158.5, 140.0)
- added R130: RC0805FR-07100KL, Resistor_SMD:R_0805_2012Metric, F.Cu at (166.5, 108.0)
- added R131: RC0805FR-071ML, Resistor_SMD:R_0805_2012Metric, F.Cu at (161.5, 84.0)
- added R132: RC0805FR-071ML, Resistor_SMD:R_0805_2012Metric, F.Cu at (166.5, 83.5)
- added R70: 470R, Resistor_SMD:R_0805_2012Metric, F.Cu at (99.0, 55.5)
- added R71: 10k, Resistor_SMD:R_0805_2012Metric, B.Cu at (200.5, 47.6)
- added R72: 47k, Resistor_SMD:R_0805_2012Metric, F.Cu at (79.5, 89.5)
- added R73: 10k, Resistor_SMD:R_0805_2012Metric, F.Cu at (81.0, 84.5)
- added R74: 10k, Resistor_SMD:R_0805_2012Metric, F.Cu at (92.0, 68.5)
- added R75: 1k, Resistor_SMD:R_0805_2012Metric, F.Cu at (95.5, 89.5)
- added R76: 470R, Resistor_SMD:R_0805_2012Metric, F.Cu at (122.5, 86.5)
- added R77: 470R, Resistor_SMD:R_0805_2012Metric, F.Cu at (117.5, 86.5)
- added R78: 10k, Resistor_SMD:R_0805_2012Metric, F.Cu at (123.5, 82.5)
- added R79: 10k, Resistor_SMD:R_0805_2012Metric, F.Cu at (120.0, 82.5)
- added R80: 10k, Resistor_SMD:R_0805_2012Metric, F.Cu at (122.5, 90.0)
- added R81: 10k, Resistor_SMD:R_0805_2012Metric, F.Cu at (110.0, 112.5)
- added R82: 12k, Resistor_SMD:R_0805_2012Metric, F.Cu at (113.5, 93.0)
- added R83: 12k, Resistor_SMD:R_0805_2012Metric, F.Cu at (109.5, 85.5)
- added R84: 20k, Resistor_SMD:R_0805_2012Metric, F.Cu at (110.5, 117.5)
- added R85: 20k, Resistor_SMD:R_0805_2012Metric, F.Cu at (128.0, 92.0)
- added R86: 470R, Resistor_SMD:R_0805_2012Metric, F.Cu at (132.0, 77.0)
- added R87: 12k, Resistor_SMD:R_0805_2012Metric, F.Cu at (127.5, 112.0)
- added R88: 12k, Resistor_SMD:R_0805_2012Metric, F.Cu at (112.0, 105.5)
- added R89: 10k, Resistor_SMD:R_0805_2012Metric, F.Cu at (110.0, 100.5)
- added R90: 5k6, Resistor_SMD:R_0805_2012Metric, F.Cu at (113.0, 96.5)
- added R91: 1M, Resistor_SMD:R_0805_2012Metric, F.Cu at (115.5, 105.5)
- added R92: 1k, Resistor_SMD:R_0805_2012Metric, F.Cu at (122.0, 117.5)
- added R93: 1k, Resistor_SMD:R_0805_2012Metric, F.Cu at (169.0, 128.5)
- added R94: 1k, Resistor_SMD:R_0805_2012Metric, F.Cu at (169.5, 124.0)
- added R95: 1k, Resistor_SMD:R_0805_2012Metric, F.Cu at (169.5, 117.0)
- added R96: 1k, Resistor_SMD:R_0805_2012Metric, F.Cu at (170.5, 120.5)
- added R97: 1k, Resistor_SMD:R_0805_2012Metric, F.Cu at (169.0, 133.5)
- added R98: 1k, Resistor_SMD:R_0805_2012Metric, F.Cu at (172.5, 131.0)
- added R99: 100k, Resistor_SMD:R_0805_2012Metric, F.Cu at (205.0, 124.0)
- added TP1: TP_PROGRAM, TestPoint:TestPoint_Pad_D1.5mm, F.Cu at (150.0, 125.0)
- added TP2: TP_ON_OFF, TestPoint:TestPoint_Pad_D1.5mm, F.Cu at (150.5, 140.0)
- added U13: BTF3050TE, Package_TO_SOT_SMD:TO-252-5_TabPin3, F.Cu at (205.5, 107.0)
- added U14: BTF3050TE, Package_TO_SOT_SMD:TO-252-5_TabPin3, F.Cu at (173.0, 108.0)
- added U15: LM74700-Q1, Package_TO_SOT_SMD:SOT-23-6, F.Cu at (78.5, 95.0)
- added U16: TPS54360B-Q1, Package_SO:HSOP-8-1EP_3.9x4.9mm_P1.27mm_EP2.41x3.1mm_ThermalVias, F.Cu at (78.5, 129.5)
- added U17: TPS7B6950-Q1, Package_TO_SOT_SMD:SOT-223-3_TabPin2, F.Cu at (91.0, 135.5)
- added U18: 74LVC1G125, Package_TO_SOT_SMD:SOT-353_SC-70-5, F.Cu at (162.0, 118.0)
- added Y1: CSTCR4M00G53-R0, Crystal:Resonator_SMD_Murata_CSTCR_4.5x2x1.15mm, F.Cu at (155.5, 125.5)
- BT1: value Battery_Cell -> ML2032; footprint 2999:BAT_2999 -> Battery:BatteryHolder_Keystone_3034_1x20mm
- C1, C21, C22, C25, C31, C37: value 0.1uF -> 100nF
- C10: value 1uF -> 1nF
- C11: value 1uF -> 0.01uF
- C12: value 0.1uF -> 1nF
- C14: value 0.1uF -> 1uF
- C15: value 270nF -> 0.1uF
- C16: value 0.1uF -> 33uF; footprint Capacitor_SMD:C_0805_2012Metric -> Capacitor_SMD:CP_Elec_6.3x7.7
- C17: value 0.22uF -> 0.1uF
- C18: value 0.22uF -> 33uF; footprint Capacitor_SMD:C_0805_2012Metric -> Capacitor_SMD:CP_Elec_6.3x7.7
- C19: value 270nF -> 100n
- C20: value 0.1uF -> 100n
- C23, C24: value 0.22uF -> 100nF
- C26: value 100uF -> 1nF; footprint Capacitor_SMD:C_1206_3216Metric -> Capacitor_SMD:C_0805_2012Metric
- C27: value 0.22uF -> 10nF
- C28, C29: value 0.01uF -> 10nF
- C30: value 100uF -> 100nF; footprint Capacitor_SMD:CP_Elec_6.3x7.7 -> Capacitor_SMD:C_0805_2012Metric
- C32, C34: value 47uF -> 100nF; footprint Capacitor_Tantalum_SMD:CP_EIA-3528-21_Kemet-B -> Capacitor_SMD:C_0805_2012Metric
- C33: value 0.1uF -> 10nF
- C35, C36: value 33uF -> 100nF; footprint Capacitor_SMD:CP_Elec_6.3x7.7 -> Capacitor_SMD:C_0805_2012Metric
- C4: value 0.01uF -> 4.7nF
- C5: value 4700pF -> 10uF; footprint Capacitor_SMD:C_0805_2012Metric -> Capacitor_SMD:C_1206_3216Metric
- C6: value 1nF -> 100nF 100V; footprint Capacitor_SMD:C_0805_2012Metric -> Capacitor_SMD:C_1206_3216Metric
- C7: value 0.01uF -> 100nF
- C8: value 1nF -> 470pF
- C9: value 0.1uF -> 470pF
- D10, D11, D12, D13: value LED -> D; footprint LED_SMD:LED_0805_2012Metric -> Diode_SMD:D_SOD-323
- D14: value 1N4148WT -> LED; footprint Diode_SMD:D_SOD-523 -> LED_SMD:LED_0805_2012Metric
- D15, D8, D9: value D -> LED; footprint Diode_SMD:D_SOD-323 -> LED_SMD:LED_0805_2012Metric
- D16, D19, D20, D21, D23, D6, D7: value D -> BAV199; footprint Diode_SMD:D_SOD-323 -> Package_TO_SOT_SMD:SOT-23
- D17: value D_Schottky -> BAV199; footprint Diode_SMD:D_PowerDI-123 -> Package_TO_SOT_SMD:SOT-23
- D18, D4, D5: value LED -> BAV199; footprint LED_SMD:LED_0805_2012Metric -> Package_TO_SOT_SMD:SOT-23
- D2: value LED -> SMAJ5.0A; footprint LED_SMD:LED_0805_2012Metric -> Diode_SMD:D_SMA
- D22: value D -> 3V6 1W (SMA); footprint Diode_SMD:D_SOD-323 -> Diode_SMD:D_SMA
- D24: value D_TVS -> BAV199; footprint Diode_SMD:D_SMB -> Package_TO_SOT_SMD:SOT-23
- D25: value D_Schottky -> BAV199; footprint Diode_SMD:D_SMA_Handsoldering -> Package_TO_SOT_SMD:SOT-23
- D26, D27, D28: value LED -> BAV199; footprint LED_SMD:LED_0805_2012Metric_Pad1.15x1.40mm_HandSolder -> Package_TO_SOT_SMD:SOT-23
- D3: value LED -> NUP2105L; footprint LED_SMD:LED_0805_2012Metric -> Package_TO_SOT_SMD:SOT-23
- F1: value Polyfuse -> 150mA
- F2: value Polyfuse -> 3A / 63V; footprint Fuse:Fuse_0603_1608Metric -> Fuse:Fuse_1206_3216Metric
- IC5: value ZXMS6006DT8 -> LD1117S33; footprint ZXMS6006DT8TA:SOT153P700X170-8N -> Package_TO_SOT_SMD:SOT-223-3_TabPin2
- Q1: value Q_DUAL_NMOS_S1G1D2S2G2D1 -> ISL9V5036P3-F085; footprint Package_TO_SOT_SMD:SOT-363_SC-70-6 -> ISL9V5036P3-F085:TO254P470X1016X2019-3P
- Q5: value ISL9V5036P3-F085 -> BSS138; footprint ISL9V5036P3-F085:TO254P470X1016X2019-3P -> Package_TO_SOT_SMD:SOT-23
- Q6: value Q_DUAL_NMOS_S1G1D2S2G2D1 -> SQM120N06-3M5L; footprint Package_TO_SOT_SMD:SOT-363_SC-70-6 -> Package_TO_SOT_SMD:TO-263-2
- R10, R21, R22: value 33 -> 0R DNP
- R11: value 33 -> 0R
- R12, R14: value 1k -> 470R
- R13, R19, R20: value 1k -> 0R
- R15: value 1k -> 10k DNP
- R16: value 10k -> 10k DNP
- R2: value 0R -> 10k
- R23: value 604R -> 10k; footprint Resistor_SMD:R_0805_2012Metric -> Resistor_SMD:R_1206_3216Metric
- R24: value 3.88k -> 10k; footprint Resistor_SMD:R_0805_2012Metric_Pad1.20x1.40mm_HandSolder -> Resistor_SMD:R_1206_3216Metric
- R25: value 0 -> 10k; footprint Resistor_SMD:R_0805_2012Metric -> Resistor_SMD:R_1206_3216Metric
- R26: value 470R -> 10k; footprint Resistor_SMD:R_0805_2012Metric -> Resistor_SMD:R_1206_3216Metric
- R27: value 2.4k -> 10k
- R28: value 470R -> 33
- R29: value 1k -> 33
- R3: value 120R -> 10k
- R30: value 2.49k -> 20m; footprint Resistor_SMD:R_0805_2012Metric -> Resistor_SMD:R_2512_6332Metric
- R31: value 2.49k -> 10k
- R32: value 0 -> 10k
- R33, R34: value 470R -> 10k
- R35: value 180k -> 10k
- R36: value 180k -> 18k; footprint Resistor_SMD:R_0805_2012Metric -> Resistor_SMD:R_1206_3216Metric
- R37, R38, R42, R43: value 348k -> 18k; footprint Resistor_SMD:R_0805_2012Metric -> Resistor_SMD:R_1206_3216Metric
- R39: value 470R -> 18k; footprint Resistor_SMD:R_0805_2012Metric -> Resistor_SMD:R_1206_3216Metric
- R4, R5: value 1k -> 10k
- R40, R41: value 180k -> 1k
- R44, R45: value 1k -> 18k; footprint Resistor_SMD:R_0805_2012Metric -> Resistor_SMD:R_1206_3216Metric
- R46: value 1k -> 4.02k
- R47: value 180k -> 4.02k
- R48: value 348k -> 4.02k
- R49: value 1k -> 4.02k; footprint Resistor_SMD:R_0805_2012Metric_Pad1.20x1.40mm_HandSolder -> Resistor_SMD:R_0805_2012Metric
- R50: value 1k -> 100k; footprint Resistor_SMD:R_0805_2012Metric_Pad1.20x1.40mm_HandSolder -> Resistor_SMD:R_0805_2012Metric
- R53, R54: value 100k -> 33; footprint Resistor_SMD:R_0805_2012Metric_Pad1.20x1.40mm_HandSolder -> Resistor_SMD:R_0805_2012Metric
- R55, R56: value 100k -> 2k49
- R57: value 1k -> 2k2
- R58: value 10k -> 470R
- R59, R60, R61, R62: value 1k -> 470R; footprint Resistor_SMD:R_0805_2012Metric_Pad1.20x1.40mm_HandSolder -> Resistor_SMD:R_0805_2012Metric
- R6, R7: value 10k -> 60.4R; footprint Resistor_SMD:R_1206_3216Metric -> Resistor_SMD:R_0805_2012Metric
- R63: value 100k -> 1k; footprint Resistor_SMD:R_0805_2012Metric_Pad1.20x1.40mm_HandSolder -> Resistor_SMD:R_0805_2012Metric
- R64, R65, R66: value 100k -> 12k; footprint Resistor_SMD:R_0805_2012Metric_Pad1.20x1.40mm_HandSolder -> Resistor_SMD:R_0805_2012Metric
- R67: value 1k -> 20k
- R68, R69: value 470R -> 20k
- R8: footprint Resistor_SMD:R_1206_3216Metric -> Resistor_SMD:R_0805_2012Metric
- R9: value 10k -> 0R DNP; footprint Resistor_SMD:R_1206_3216Metric -> Resistor_SMD:R_0805_2012Metric
- U10: value SP720 -> LMV324; footprint Package_SO:SOIC-16_3.9x9.9mm_P1.27mm -> Package_SO:SOIC-14_3.9x8.7mm_P1.27mm
- U11: value LMV324LIDT -> LMV324
- U12: value MC78M05_TO252 -> DRV8434A; footprint Package_TO_SOT_SMD:TO-252-2 -> Package_SO:HTSSOP-28-1EP_4.4x9.7mm_P0.65mm_EP2.85x5.4mm_ThermalVias
- U6: value TC4424A -> USBLC6-2SC6; footprint Package_SO:SOIC-8_3.9x4.9mm_P1.27mm -> Package_TO_SOT_SMD:SOT-23-6
- U8: value TC4424A -> TPS3823-33DBV; footprint Package_SO:SOIC-8_3.9x4.9mm_P1.27mm -> Package_TO_SOT_SMD:SOT-23-5
- U9: value LMV324LIDT -> 74LVC1G00; footprint Package_SO:SOIC-14_3.9x8.7mm_P1.27mm -> Package_TO_SOT_SMD:SOT-353_SC-70-5
- moved Q1 129.5 mm to (196.1, 60.1), turned to 90 degrees
- moved R29 127.2 mm to (199.2, 65.1)
- moved C4 123.6 mm to (192.5, 99.0)
- moved R66 123.4 mm to (77.0, 85.5), turned to 0 degrees
- moved R65 122.8 mm to (82.5, 75.5), turned to 0 degrees
- moved IC5 121.3 mm to (77.0, 119.5), turned to 90 degrees
- moved R28 119.6 mm to (193.7, 65.1), turned to 0 degrees
- moved C18 119.0 mm to (183.0, 105.5), turned to 0 degrees
- moved R30 117.3 mm to (207.0, 92.0), turned to 90 degrees
- moved D22 116.6 mm to (73.5, 89.5), turned to 0 degrees
- moved C5 116.5 mm to (161.5, 64.0), turned to 0 degrees
- moved R61 112.5 mm to (106.0, 54.5)
- moved R31 112.0 mm to (209.5, 57.5)
- moved R62 110.4 mm to (102.5, 54.5)
- moved C19 110.0 mm to (176.0, 84.0), turned to 0 degrees
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Connections:
- net /Conntectors/Diagnose Stecker renamed DIAG-IN
- net /Conntectors/Tacho Data renamed TACHO-DATA
- C1 pad 1: +3V3 -> T_3V3
- C10 pad 1: +5V -> Net-(IC1-IN1+)
- C10 pad 2: GND -> Net-(IC1-IN1-)
- C11 pad 1: IGN_V+ -> +5V
- C12 pad 1: IGN_V+ -> Net-(IC1-IN2-)
- C12 pad 2: GND -> Net-(IC1-IN2+)
- C13 pad 1: O2_Sensor -> +5V
- C14 pad 1: Net-(C14-Pad1) -> +5V
- C15 pad 1: ADC-Clamp-5 -> GND
- C15 pad 2: GND -> +3V3
- C16 pad 1: GND -> +3V3
- C16 pad 2: MAP-5V -> GND
- C17 pad 1: O2-5V -> 12V-PROT
- C18 pad 1: ADC-Clamp-7 -> 12V-PROT
- C19 pad 1: ADC-Clamp-6 -> +3V3
- C2 pad 1: GND -> +3V3
- C2 pad 2: +5V -> GND
- C20 pad 1: IAT_Sensor -> +3V3
- C21 pad 1: CLT_Sensor -> Net-(C21-Pad1)
- C22 pad 1: GND -> Net-(C22-Pad1)
- C22 pad 2: BARO-5V -> GND
- C23 pad 1: ADC-Clamp-11 -> Net-(C23-Pad1)
- C24 pad 1: ADC-Clamp-12 -> MCU-A4
- C25 pad 1: TPS_Sensor -> MCU-A5
- C26 pad 1: GND -> MCU-A14
- C26 pad 2: +3V3 -> GND
- C27 pad 1: TPS-5V -> MCU-A0
- C28 pad 1: GND -> MCU-A1
- C28 pad 2: MCU-D35 -> GND
- C29 pad 1: GND -> MCU-A2
- C29 pad 2: MCU-D34 -> GND
- C3 pad 2: MCU-D21 -> +5V
- C30 pad 1: Net-(A1-VMOT) -> Net-(U10A-+)
- C31 pad 1: +5V -> MCU-D33
- C32 pad 1: +5V -> MCU-A15
- C33 pad 1: +5V -> MCU-A3
- C34 pad 1: +5V -> +3V3
- C35 pad 1: 12V-PROT -> Net-(C35-Pad1)
- C36 pad 1: 12V-PROT -> Net-(C36-Pad1)
- C37 pad 1: 12V-PROT -> MCU-D4
- C4 pad 1: GND -> Net-(C4-Pad1)
- C4 pad 2: Net-(JP4-B) -> GND
- C5 pad 1: Net-(JP5-B) -> /Conntectors/VDDA-J2
- C5 pad 2: GND -> GNDA
- C6 pad 1: Net-(IC1-IN1+) -> 12V-SW
- C6 pad 2: Net-(IC1-IN1-) -> GND
- C7 pad 1: +5V -> USB 5V
- C8 pad 1: Net-(IC1-IN2-) -> MCU-D20
- C8 pad 2: Net-(IC1-IN2+) -> GND
- C9 pad 1: +5V -> MCU-D21
- D1 pad 1: +3V3 -> Net-(D1-K)
- D1 pad 2: Net-(D1-A) -> +3V3
- D10 pad 1: Net-(D10-K) -> INJ2
- D11 pad 1: Net-(D11-K) -> INJ1
- D12 pad 1: GND -> INJ4
- D13 pad 1: GND -> INJ3
- D14 pad 1: Clutch_in -> Net-(D12-A)
- D14 pad 2: ADC-Clamp-6 -> Net-(D14-A)
- D15 pad 1: 12V-SW -> Net-(D13-A)
- D15 pad 2: IDLE-OUT -> Net-(D15-A)
- D16 pad 1: 12V-SW -> GND
- D16 pad 2: SPARE2-OUT -> +3V3
- D17 pad 1: Net-(A1-VMOT) -> GND
- D17 pad 2: 12V-SW -> +3V3
- D18 pad 1: FUELPUMP-OUT -> GND
- D18 pad 2: Net-(D18-A) -> +3V3
- D19 pad 1: 12V-SW -> GND
- D19 pad 2: FUELPUMP-OUT -> +3V3
- D2 pad 1: GND -> /Conntectors/VDDA-J2
- D2 pad 2: Net-(D2-A) -> GNDA
- D20 pad 1: 12V-SW -> GND
- D20 pad 2: FAN-OUT -> +3V3
- D21 pad 1: 12V-SW -> GND
- D21 pad 2: BOOST-OUT -> +3V3
- D22 pad 1: 12V-SW -> +3V3
- D22 pad 2: SPARE1-OUT -> GND
- D23 pad 1: 12V-SW -> GND
- D23 pad 2: SPARE2_OUT -> +3V3
- D24 pad 1: 12V-PROT -> GND
- D24 pad 2: GND -> +3V3
- D25 pad 1: 12V-PROT -> GND
- D25 pad 2: 12V-SW -> +3V3
- D26 pad 2: Net-(D26-A) -> +3V3
- D27 pad 2: Net-(D27-A) -> +3V3
- D28 pad 2: Net-(D28-A) -> +3V3
- D3 pad 1: GND -> CAN_L
- D3 pad 2: Net-(D3-A) -> CAN_H
- D4 pad 1: Net-(D4-K) -> GND
- D4 pad 2: Net-(D4-A) -> +3V3
- D5 pad 1: Net-(D5-K) -> GND
- D5 pad 2: Net-(D5-A) -> +3V3
- D6 pad 1: INJ2 -> GND
- D6 pad 2: Net-(D4-K) -> +3V3
- D7 pad 1: INJ3 -> GND
- D7 pad 2: Net-(D5-K) -> +3V3
- D8 pad 1: INJ1 -> Net-(D10-A)
- D8 pad 2: Net-(D10-K) -> Net-(D8-A)
- D9 pad 1: INJ4 -> Net-(D11-A)
- D9 pad 2: Net-(D11-K) -> Net-(D9-A)
- F1 pad 1: Net-(SW3-NO_1) -> VDDA
- F1 pad 2: +5V -> /Conntectors/VDDA-J2
- F2 pad 1: +5V -> 12V-SW
- F2 pad 2: VDDA -> /Power Regulator/VBAT_F
- IC1 pad 4: MCU-D20 -> VR1-OUT
- IC1 pad 5: MCU-D21 -> VR2-OUT
- IC2 pad 1: Net-(IC2-INPUT_1) -> /Outputs/G_FI
- IC2 pad 2: GND -> PGND
- IC2 pad 3: Net-(IC2-INPUT_2) -> /Outputs/G_STRT
- IC2 pad 4: GND -> PGND
- IC2 pad 5: SPARE2-OUT -> STARTER-OUT
- IC2 pad 6: SPARE2-OUT -> STARTER-OUT
- IC2 pad 7: IDLE-OUT -> FI-LAMP
- IC2 pad 8: IDLE-OUT -> FI-LAMP
- IC3 pad 1: Net-(IC3-INPUT_1) -> /Outputs/G_FUEL
- IC3 pad 2: GND -> PGND
- IC3 pad 3: Net-(IC3-INPUT_2) -> /Outputs/G_TACH
- IC3 pad 4: GND -> PGND
- IC4 pad 1: Net-(IC4-INPUT_1) -> /Outputs/G_FAN
- IC4 pad 2: GND -> PGND
- IC4 pad 3: Net-(IC4-INPUT_2) -> /Outputs/G_SPARE
- IC4 pad 4: GND -> PGND
- IC4 pad 5: SPARE2_OUT -> SPARE-OUT
- IC4 pad 6: SPARE2_OUT -> SPARE-OUT
- IC4 pad 7: SPARE1-OUT -> FAN-OUT
- IC4 pad 8: SPARE1-OUT -> FAN-OUT
- IC5 pad 1: Net-(IC5-INPUT_1) -> GND
- IC5 pad 2: GND -> +3V3
- IC5 pad 3: Net-(IC5-INPUT_2) -> +5V
- J2 pad 18: GND -> PGND
- J2 pad 20: /Conntectors/Neutral input -> NEUTRAL-IN
- J2 pad 21: GND -> PGND
- J2 pad 23: USB D- -> /Conntectors/USB-J2-D-
- J2 pad 24: USB GND -> GND
- J2 pad 25: USB D+ -> /Conntectors/USB-J2-D+
- J2 pad 28: /Conntectors/Starter Relay FB -> STARTER-OUT
- J2 pad 31: SPARE1-OUT -> STEPPER-A1
- J2 pad 32: SPARE2-OUT -> STEPPER-A2
- J2 pad 33: unconnected-(J2-Pad33) -> Knock-Sensor-1
- J2 pad 34: unconnected-(J2-Pad34) -> Knock-Sensor-2
- J2 pad 39: ADC-Clamp-5 -> Flex_Sensor
- J2 pad 42: /Conntectors/FI FB -> FI-LAMP
- J2 pad 45: O2-Heater -> STEPPER-B2
- J2 pad 46: unconnected-(J2-Pad46) -> O2-HEATER
- J2 pad 47: unconnected-(J2-Pad47) -> SPARE-OUT
- J2 pad 48: VDDA -> /Conntectors/VDDA-J2
- J2 pad 54: GND -> GNDA
- J2 pad 8: IDLE-OUT -> STEPPER-B1
- Q1 pad 1: MCU-D20 -> /Drivers/G_IGN2
- Q1 pad 2: +3V3 -> IGN2
- Q1 pad 3: Net-(JP3-B) -> /Drivers/IGBT_E
- Q2 pad 1: Net-(Q2-Pad1) -> /Drivers/G_IGN1
- Q2 pad 3: GND -> /Drivers/IGBT_E
- Q3 pad 1: Net-(Q3-Pad1) -> /Drivers/G_IGN3
- Q3 pad 2: IGN2 -> IGN3
- Q3 pad 3: GND -> /Drivers/IGBT_E
- Q4 pad 1: Net-(Q4-Pad1) -> /Drivers/G_IGN4
- Q4 pad 2: IGN3 -> IGN4
- Q4 pad 3: GND -> /Drivers/IGBT_E
- Q5 pad 1: Net-(Q5-Pad1) -> /Outputs/OUT-FAULT-H
- Q5 pad 2: IGN4 -> MCU-D9
- Q6 pad 1: MCU-D35 -> /Power Regulator/ID_GATE
- Q6 pad 2: +3V3 -> /Power Regulator/VBAT_ID
- Q6 pad 3: SPARE2-Digital -> /Power Regulator/VBAT_F
- R1 pad 2: Net-(D1-A) -> Net-(D1-K)
- R10 pad 1: Net-(Q2-Pad1) -> CAM-IN+
- R10 pad 2: Net-(U6-OUT_B) -> Net-(R10-Pad2)
- R11 pad 1: Net-(Q3-Pad1) -> CRANK-IN+
- R11 pad 2: Net-(U6-OUT_A) -> VR1-IN+
- R12 pad 1: Net-(D2-A) -> /Crank and Cam/CRANK-SIG
- R12 pad 2: Net-(U6-OUT_B) -> MCU-D20
- R13 pad 1: Net-(D3-A) -> CAM-IN+
- R13 pad 2: Net-(U6-OUT_A) -> VR2-IN+
- R14 pad 1: Net-(D4-A) -> /Crank and Cam/CAM-SIG
- R14 pad 2: 12V-SW -> MCU-D21
- R15 pad 1: 12V-SW -> /Crank and Cam/CRANK-HALL
- R15 pad 2: Net-(D5-A) -> +3V3
- R16 pad 1: OUTEN_1 -> /Crank and Cam/CAM-HALL
- R16 pad 2: GND -> +3V3
- R17 pad 1: Net-(D10-A) -> Net-(R17-Pad1)
- R17 pad 2: 12V-SW -> /Crank and Cam/CRANK-HALL
- R18 pad 1: Net-(D11-A) -> Net-(R10-Pad2)
- R18 pad 2: 12V-SW -> /Crank and Cam/CAM-HALL
- R19 pad 1: Net-(D12-A) -> VR1-OUT
- R19 pad 2: Net-(U8-OUT_A) -> /Crank and Cam/CRANK-SIG
- R2 pad 1: GND -> +3V3
- R2 pad 2: Net-(U3-STBY) -> MCU-D6
- R20 pad 1: Net-(D13-A) -> VR2-OUT
- R20 pad 2: Net-(U8-OUT_B) -> /Crank and Cam/CAM-SIG
- R21 pad 1: Net-(Q4-Pad1) -> /Crank and Cam/CRANK-HALL
- R21 pad 2: Net-(U8-OUT_A) -> /Crank and Cam/CRANK-SIG
- R22 pad 1: Net-(Q5-Pad1) -> /Crank and Cam/CAM-HALL
- R22 pad 2: Net-(U8-OUT_B) -> /Crank and Cam/CAM-SIG
- R23 pad 1: GND -> VR1-IN+
- R23 pad 2: Net-(C14-Pad1) -> Net-(IC1-IN1+)
- R24 pad 1: Net-(C14-Pad1) -> CRANK-IN-
- R24 pad 2: 12V-SW -> Net-(IC1-IN1-)
- R25 pad 1: Map_Sensor -> CAM-IN-
- R25 pad 2: MAP-5V -> Net-(IC1-IN2-)
- R26 pad 1: O2-5V -> VR2-IN+
- R26 pad 2: O2_Sensor -> Net-(IC1-IN2+)
- R27 pad 1: +3V3 -> MC33810_1-CS
- R27 pad 2: ADC-Clamp-5 -> +3V3
- R28 pad 1: ADC-Clamp-7 -> /Drivers/G_IGN2
- R28 pad 2: Net-(C14-Pad1) -> T_IGN2
- R29 pad 1: ADC-Clamp-6 -> /Drivers/G_IGN1
- R29 pad 2: +3V3 -> T_IGN1
- R3 pad 1: CAN_L -> GND
- R3 pad 2: Net-(JP1-Pad2) -> Net-(U3-STBY)
- R30 pad 1: IAT_Sensor -> /Drivers/IGBT_E
- R30 pad 2: +3V3 -> PGND
- R31 pad 1: CLT_Sensor -> /Drivers/G_IGN1
- R31 pad 2: +3V3 -> /Drivers/IGBT_E
- R32 pad 1: Baro_Sensor -> /Drivers/G_IGN2
- R32 pad 2: BARO-5V -> /Drivers/IGBT_E
- R33 pad 1: ADC-Clamp-11 -> /Drivers/G_IGN3
- R33 pad 2: IAT_Sensor -> /Drivers/IGBT_E
- R34 pad 1: ADC-Clamp-12 -> /Drivers/G_IGN4
- R34 pad 2: CLT_Sensor -> /Drivers/IGBT_E
- R35 pad 1: Net-(U9A-+) -> OUTEN_1
- R35 pad 2: BARO-5V -> +3V3
- R36 pad 1: Net-(U9C-+) -> IGN1
- R36 pad 2: O2-5V -> Net-(R36-Pad2)
- R37 pad 1: GND -> IGN2
- R37 pad 2: Net-(U9A-+) -> Net-(R37-Pad2)
- R38 pad 1: GND -> IGN3
- R38 pad 2: Net-(U9C-+) -> Net-(R38-Pad2)
- R39 pad 1: TPS-5V -> IGN4
- R39 pad 2: TPS_Sensor -> Net-(R39-Pad2)
- R4 pad 1: MCU-D20 -> +3V3
- R4 pad 2: +3V3 -> Net-(U2-IO2)
- R40 pad 1: Net-(U9B-+) -> Net-(D8-A)
- R40 pad 2: MAP-5V -> 12V-PROT
- R41 pad 1: Net-(U9D-+) -> 12V-PROT
- R41 pad 2: TPS-5V -> Net-(D9-A)
- R42 pad 1: GND -> Net-(R36-Pad2)
- R42 pad 2: Net-(U9B-+) -> /Drivers/FB0
- R43 pad 1: GND -> Net-(R37-Pad2)
- R43 pad 2: Net-(U9D-+) -> /Drivers/FB1
- R44 pad 1: MCU-D35 -> Net-(R38-Pad2)
- R44 pad 2: +3V3 -> /Drivers/FB2
- R45 pad 1: +5V -> Net-(R39-Pad2)
- R45 pad 2: Gear_Position -> /Drivers/FB3
- R46 pad 1: MCU-D34 -> /Drivers/FB0
- R46 pad 2: +3V3 -> PGND
- R47 pad 1: Net-(U11B-+) -> /Drivers/FB1
- R47 pad 2: SPARE2_Sensor -> PGND
- R48 pad 1: GND -> /Drivers/FB2
- R48 pad 2: Net-(U11B-+) -> PGND
- R49 pad 1: Net-(IC2-INPUT_1) -> /Drivers/FB3
- R49 pad 2: MCU-D27 -> PGND
- R5 pad 2: MCU-D21 -> Net-(U2-IO3)
- R50 pad 1: Net-(IC2-INPUT_2) -> MCU-D2
- R50 pad 2: MCU-D26 -> GND
- R51 pad 1: Net-(IC3-INPUT_1) -> Net-(D14-A)
- R51 pad 2: MCU-D5 -> 12V-PROT
- R52 pad 1: Net-(IC3-INPUT_2) -> Net-(D15-A)
- R52 pad 2: MCU-D8 -> 12V-PROT
- R53 pad 1: GND -> /Drivers/G_IGN3
- R53 pad 2: Net-(IC2-INPUT_1) -> T_IGN3
- R54 pad 1: GND -> /Drivers/G_IGN4
- R54 pad 2: Net-(IC2-INPUT_2) -> T_IGN4
- R55 pad 1: Net-(IC3-INPUT_1) -> +3V3
- R55 pad 2: GND -> IAT_Sensor
- R56 pad 1: GND -> +3V3
- R56 pad 2: Net-(IC3-INPUT_2) -> CLT_Sensor
- R57 pad 1: 12V-SW -> +3V3
- R57 pad 2: Net-(D18-A) -> Flex_Sensor
- R58 pad 1: TACHO-OUT -> Map_Sensor
- R58 pad 2: 12V-SW -> Net-(C21-Pad1)
- R59 pad 1: Net-(IC4-INPUT_1) -> Baro_Sensor
- R59 pad 2: MCU-D29 -> Net-(C22-Pad1)
- R6 pad 1: VR1-IN+ -> CAN_H
- R6 pad 2: Net-(IC1-IN1+) -> Net-(C4-Pad1)
- R60 pad 1: Net-(IC4-INPUT_2) -> TPS_Sensor
- R60 pad 2: MCU-D28 -> Net-(C23-Pad1)
- R61 pad 1: Net-(IC5-INPUT_1) -> IAT_Sensor
- R61 pad 2: MCU-D25 -> MCU-A4
- R62 pad 1: Net-(IC5-INPUT_2) -> CLT_Sensor
- R62 pad 2: MCU-D24 -> MCU-A5
- R63 pad 1: Net-(IC4-INPUT_1) -> Flex_Sensor
- R63 pad 2: GND -> MCU-A14
- R64 pad 1: GND -> Net-(C21-Pad1)
- R64 pad 2: Net-(IC4-INPUT_2) -> MCU-A0
- R65 pad 1: Net-(IC5-INPUT_1) -> Net-(C22-Pad1)
- R65 pad 2: GND -> MCU-A1
- R66 pad 1: GND -> Net-(C23-Pad1)
- R66 pad 2: Net-(IC5-INPUT_2) -> MCU-A2
- R67 pad 1: 12V-SW -> MCU-A0
- R67 pad 2: Net-(D26-A) -> GNDA
- R68 pad 1: +5V -> MCU-A1
- R68 pad 2: Net-(D27-A) -> GNDA
- R69 pad 1: VDDA -> MCU-A2
- R69 pad 2: Net-(D28-A) -> GNDA
- R7 pad 1: CRANK-IN- -> Net-(C4-Pad1)
- R7 pad 2: Net-(IC1-IN1-) -> CAN_L
- R8 pad 1: CAM-IN- -> +3V3
- R8 pad 2: Net-(IC1-IN2-) -> MCU-D7
- R9 pad 1: VR2-IN+ -> CRANK-IN+
- R9 pad 2: Net-(IC1-IN2+) -> Net-(R17-Pad1)
- U1 pad 15: +3V3 -> T_3V3
- U1 pad 25: unconnected-(U1-33_MCLK2-Pad25) -> MCU-D33
- U1 pad 28: ADC-Clamp-6 -> MCU-D36
- U1 pad 29: unconnected-(U1-37_CS-Pad29) -> MCU-D37
- U1 pad 30: ADC-Clamp-5 -> MCU-A14
- U1 pad 31: ADC-Clamp-7 -> MCU-A15
- U1 pad 32: ADC-Clamp-4 -> MCU-A16
- U1 pad 33: ADC-Clamp-3 -> MCU-A17
- U1 pad 36: ADC-Clamp-11 -> MCU-A0
- U1 pad 37: ADC-Clamp-12 -> MCU-A1
- U1 pad 38: ADC-Clamp-13 -> MCU-A2
- U1 pad 39: ADC-Clamp-14 -> MCU-A3
- U1 pad 4: MC33814-CS -> MCU-D2
- U1 pad 46: +3V3 -> T_3V3
- U1 pad 51: +3V3 -> T_3V3
- U1 pad 53: PROG -> Net-(U1-PROGRAM)
- U1 pad 54: RESET -> Net-(U1-ON_OFF)
- U1 pad 55: USB 5V -> unconnected-(U1-5V-Pad55)
- U1 pad 56: USB D- -> unconnected-(U1-D--Pad56)
- U1 pad 57: USB D+ -> unconnected-(U1-D+-Pad57)
- U1 pad 58: USB GND -> unconnected-(U1-GND-Pad58)
- U1 pad 66: unconnected-(U1-D--Pad66) -> USB D-
- U1 pad 67: unconnected-(U1-D+-Pad67) -> USB D+
- U10 pad 1: ADC-Clamp-1 -> Net-(U10A--)
- U10 pad 10: ADC-Clamp-9 -> GND
- U10 pad 11: ADC-Clamp-10 -> GND
- U10 pad 12: ADC-Clamp-11 -> GND
- U10 pad 13: ADC-Clamp-12 -> Net-(U10D--)
- U10 pad 14: ADC-Clamp-13 -> Net-(U10D--)
- U10 pad 2: ADC-Clamp-2 -> Net-(U10A--)
- U10 pad 3: ADC-Clamp-3 -> Net-(U10A-+)
- U10 pad 4: ADC-Clamp-4 -> +3V3
- U10 pad 5: ADC-Clamp-5 -> GND
- U10 pad 6: ADC-Clamp-6 -> Net-(U10B--)
- U10 pad 7: ADC-Clamp-7 -> Net-(U10B--)
- U10 pad 8: GND -> Net-(U10C--)
- U10 pad 9: ADC-Clamp-8 -> Net-(U10C--)
- U11 pad 1: ADC-Clamp-4 -> Net-(R91-Pad2)
- U11 pad 10: unconnected-(U11C-+-Pad10) -> GND
- U11 pad 12: unconnected-(U11D-+-Pad12) -> GND
- U11 pad 2: ADC-Clamp-4 -> Net-(U11A--)
- U11 pad 3: Gear_Position -> Net-(D30-K1A2)
- U11 pad 4: VDDA -> +3V3
- U11 pad 5: Net-(U11B-+) -> GND
- U11 pad 6: ADC-Clamp-3 -> Net-(U11B--)
- U11 pad 7: ADC-Clamp-3 -> Net-(U11B--)
- U12 pad 1: 12V-PROT -> Net-(U12-VCP)
- U12 pad 2: GND -> 12V-PROT
- U12 pad 3: +5V -> PGND
- U2 pad 3: +3V3 -> Net-(U2-IO2)
- U2 pad 7: +3V3 -> Net-(U2-IO3)
- U6 pad 1: unconnected-(U6-NC-Pad1) -> /Conntectors/USB-J2-D-
- U6 pad 2: Net-(U6-IN_A) -> GND
- U6 pad 3: GND -> /Conntectors/USB-J2-D+
- U6 pad 4: Net-(U6-IN_B) -> USB D+
- U6 pad 5: Net-(U6-OUT_B) -> USB 5V
- U6 pad 6: IGN_V+ -> USB D-
- U7 pad 1: INJ3 -> INJ1
- U7 pad 14: Net-(U6-IN_A) -> T_IGN2
- U7 pad 15: unconnected-(U7-FB1-Pad15) -> /Drivers/FB1
- U7 pad 17: INJ1 -> INJ4
- U7 pad 18: unconnected-(U7-FB3-Pad18) -> /Drivers/FB3
- U7 pad 19: Net-(U7-GD3) -> T_IGN4
- U7 pad 2: unconnected-(U7-FB0-Pad2) -> /Drivers/FB0
- U7 pad 25: 12V-SW -> 12V-PROT
- U7 pad 26: unconnected-(U7-RSP-Pad26) -> /Drivers/IGBT_E
- U7 pad 27: unconnected-(U7-RSN-Pad27) -> PGND
- U7 pad 3: Net-(U6-IN_B) -> T_IGN1
- U7 pad 30: Net-(U7-GD2) -> T_IGN3
- U7 pad 31: unconnected-(U7-FB2-Pad31) -> /Drivers/FB2
- U7 pad 32: INJ4 -> INJ3
- U7 pad 33: GND -> PGND
- U8 pad 1: unconnected-(U8-NC-Pad1) -> /Drivers/WDT-RESET
- U8 pad 2: Net-(U7-GD2) -> GND
- U8 pad 3: GND -> +3V3
- U8 pad 4: Net-(U7-GD3) -> MCU-D3
- U8 pad 5: Net-(U8-OUT_B) -> +3V3
- U9 pad 1: MCU-A4 -> MCU-D2
- U9 pad 2: MCU-A4 -> /Drivers/WDT-RESET
- U9 pad 3: Net-(U9A-+) -> GND
- U9 pad 4: VDDA -> OUTEN_1
- U9 pad 5: Net-(U9B-+) -> +3V3
Routing:
- net GND: track 22.6 -> 1367.6 mm, vias 176 -> 12
- net 12V-PROT: track 32.8 -> 565.9 mm, vias 0 -> 15
- net PGND: track 0.00 -> 444.5 mm, vias 0 -> 21
- net +3V3: track 444.8 -> 729.9 mm, vias 19 -> 31
- net MCU-D33: track 0.00 -> 281.4 mm, vias 0 -> 4
- net Knock-Sensor-1: track 0.00 -> 255.2 mm, vias 0 -> 5
- net ADC-Clamp-5: track 227.2 -> 0.00 mm, vias 4 -> 0
- net ADC-Clamp-6: track 223.3 -> 0.00 mm, vias 2 -> 0
- net ADC-Clamp-4: track 212.4 -> 0.00 mm, vias 4 -> 0
- net GNDA: track 0.00 -> 211.3 mm, vias 0 -> 3
- net ADC-Clamp-7: track 202.7 -> 0.00 mm, vias 2 -> 0
- net ADC-Clamp-12: track 202.4 -> 0.00 mm, vias 6 -> 0
- net 12V-SW: track 376.2 -> 185.5 mm, vias 11 -> 4
- net ADC-Clamp-3: track 188.5 -> 0.00 mm, vias 2 -> 0
- net ADC-Clamp-11: track 177.7 -> 0.00 mm, vias 4 -> 0
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Other:
- board text added: "Hayabusa ECU Rev 3.0"
- board text removed: "Kontakt Author: Kevin Müller (HasiKe) Mail: kevin.mueller@hasike.de Social: @kevin_der_stein Web: www.HasiKe.de doku: www.github.com/HasiKe/Hayabusa.git"
