File: hardware/ECU/Inputs.kicad_sch (KiCad schematic)
At the start: 39 parts, among them U10 SP720, U9 LMV324LIDT

Commit message: Update ECU-Hardware, Dokumente und Explosionszeichnungen
Parts:
- removed C13, C14, C16, C20: 0.1uF, Capacitor_SMD:C_0805_2012Metric, symbol Device:C
- removed C15, C19: 270nF, Capacitor_SMD:C_0805_2012Metric, symbol Device:C
- removed C17, C18: 0.22uF, Capacitor_SMD:C_0805_2012Metric, symbol Device:C
- removed D14: 1N4148WT, Diode_SMD:D_SOD-523, symbol Diode:1N4148WT
- removed R23: 604R, Resistor_SMD:R_0805_2012Metric, symbol Device:R
- removed R24: 3.88k, Resistor_SMD:R_0805_2012Metric_Pad1.20x1.40mm_HandSolder, symbol Device:R
- removed R25, R32: 0, Resistor_SMD:R_0805_2012Metric, symbol Device:R
- removed R26, R28, R33, R34, R39: 470R, Resistor_SMD:R_0805_2012Metric, symbol Device:R
- removed R27: 2.4k, Resistor_SMD:R_0805_2012Metric, symbol Device:R
- removed R29: 1k, Resistor_SMD:R_0805_2012Metric, symbol Device:R
- removed R30, R31: 2.49k, Resistor_SMD:R_0805_2012Metric, symbol Device:R
- removed R35, R36, R40, R41: 180k, Resistor_SMD:R_0805_2012Metric, symbol Device:R
- removed R37, R38, R42, R43: 348k, Resistor_SMD:R_0805_2012Metric, symbol Device:R
- removed U10: SP720, Package_SO:SOIC-16_3.9x9.9mm_P1.27mm, symbol IC_Automotive:SP720
- removed U9: LMV324LIDT, Package_SO:SOIC-14_3.9x8.7mm_P1.27mm, symbol Amplifier_Operational:LMV324
- added C28, C29, C33: 10nF, Capacitor_SMD:C_0805_2012Metric, symbol Device:C
- added C30, C31, C32, C34: 100nF, Capacitor_SMD:C_0805_2012Metric, symbol Device:C
- added D16, D17, D18, D19, D20, D21, D23, D24, D25: BAV199, Package_TO_SOT_SMD:SOT-23, symbol Diode:BAV199
- added D22: 3V6 1W (SMA), Diode_SMD:D_SMA, symbol Device:D_Zener
- added R55, R56: 2k49, Resistor_SMD:R_0805_2012Metric, symbol Device:R
- added R57: 2k2, Resistor_SMD:R_0805_2012Metric, symbol Device:R
- added R58, R59, R60, R61, R62, R70: 470R, Resistor_SMD:R_0805_2012Metric, symbol Device:R
- added R63, R75: 1k, Resistor_SMD:R_0805_2012Metric, symbol Device:R
- added R64, R65, R66: 12k, Resistor_SMD:R_0805_2012Metric, symbol Device:R
- added R67, R68, R69: 20k, Resistor_SMD:R_0805_2012Metric, symbol Device:R
- added R71, R73, R74: 10k, Resistor_SMD:R_0805_2012Metric, symbol Device:R
- added R72: 47k, Resistor_SMD:R_0805_2012Metric, symbol Device:R
- added U10: LMV324, Package_SO:SOIC-14_3.9x8.7mm_P1.27mm, symbol Amplifier_Operational:LMV324
- C21, C22, C25: value 0.1uF -> 100nF; Supplier (none) -> DigiKey; URL https://www.digikey.com.au/product-detail/en/yageo/CC0805KR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 -> (none)
- C23, C24: value 0.22uF -> 100nF; Digikey Part Number 1276-1284-1-ND -> 311-1140-1-ND; Manufacturer_Name Samsung -> Yageo; Manufacturer_Part_Number CL21B224KOCNNNC -> CC0805KRX7R9BB104; Supplier (none) -> DigiKey; URL https://www.digikey.com/product-detail/en/samsung-electro-m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 -> (none)
- C26: value 100uF -> 1nF; footprint Capacitor_SMD:C_1206_3216Metric -> Capacitor_SMD:C_0805_2012Metric; Digikey Part Number 1276-1782-1-ND -> 399-16591-1-ND; Manufacturer_Name Samsung -> KEMET; Manufacturer_Part_Number CL31A107MQHNNNE -> C0805C102J5HACAUTO; Supplier (none) -> DigiKey; URL https://www.digikey.com.au/product-detail/en/samsung-electr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 -> (none)
- C27: value 0.22uF -> 10nF; Digikey Part Number 1276-1284-1-ND -> 311-1136-1-ND; Manufacturer_Name Samsung -> Yageo; Manufacturer_Part_Number CL21B224KOCNNNC -> CC0805KRX7R9BB103; Supplier (none) -> DigiKey; URL https://www.digikey.com/product-detail/en/samsung-electro-m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 -> (none)
Connections:
- net ADC-Clamp-12 is gone; now on net MCU-A4: C24.1
- net BARO-5V is gone; now on net GND: C22.2
- net +3V3: now also C34.1, D16.2 (K2), D17.2 (K2), D18.2 (K2), D19.2 (K2), D20.2 (K2), D21.2 (K2), D22.1 (K), D23.2 (K2), D24.2 (K2), D25.2 (K2), R55.1, R56.1, R57.1, R73.1, U10.4 (V+); no longer C26.2
- net Baro_Sensor: now also R59.1
- net CLT_Sensor: now also R56.2, R62.1; no longer C21.1
- net Clutch_in: now also R71.1
- net GND: now also C26.2, C28.2, C29.2, C30.2, C31.2, C32.2, C33.2, C34.2, D16.1 (A1), D17.1 (A1), D18.1 (A1), D19.1 (A1), D20.1 (A1), D21.1 (A1), D22.2 (A), D23.1 (A1), D24.1 (A1), D25.1 (A1), U10.10 (+), U10.11 (V-), U10.12 (+), U10.5 (+); no longer C22.1, C26.1
- net IAT_Sensor: now also R55.2, R61.1
- net MCU-A4: now also D16.3 (K1A2), R61.2
- net MCU-A5: now also C25.1, D17.3 (K1A2), R62.2
- net Map_Sensor: now also R58.1
- net O2_Sensor: now also R70.1
- net TPS_Sensor: now also R60.1; no longer C25.1
- net ADC-Clamp-11: no longer names the net of C23.1
- net ADC-Clamp-11: now also R60.2, R66.1
- net TPS-5V renamed MCU-A0
- net MCU-A0: now also D19.3 (K1A2), R64.2, R67.1
- new net: C21.1, R58.2, R64.1
- new net: C22.1, R59.2, R65.1
- new net: U10.6 (-), U10.7
- new net: U10.13 (-), U10.14
- new net: C30.1, R70.2, U10.3 (+)
- new net: U10.8, U10.9 (-)
- new net: R75.1, U10.1, U10.2 (-)
- new net 12V-PROT: R72.1
- new net Flex_Sensor: R57.2, R63.1
- new net GNDA: R67.2, R68.2, R69.2, R74.2
- new net MCU-A1: C28.1, D20.3 (K1A2), R65.2, R68.1
- new net MCU-A14: C26.1, D18.3 (K1A2), R63.2
- new net MCU-A15: C32.1, D24.3 (K1A2), R72.2, R74.1
- new net MCU-A2: C29.1, D21.3 (K1A2), R66.2, R69.1
- new net MCU-A3: C33.1, D25.3 (K1A2), R75.2
- new net MCU-D33: C31.1, D23.3 (K1A2), R71.2, R73.2
Other:
- note added: "Baro (J2.52) — ratiometrisch 5 V → 0,625"
- note added: "Batteriespannung (12V-PROT) — 47k/10k = 0,1754, 14,3 V → 2,51 V"
- note added: "CLT (J2.51) — NTC, Pullup 2k49 an +3V3"
- note added: "Clutch (J2.19) — Schalter nach Masse, Pullup 10k"
- note added: "Flex (J2.39) — Open-Collector-Frequenz, Pullup 2k2, Timer-Capture"
- note added: "IAT (J2.50) — NTC, Pullup 2k49 an +3V3"
- note added: "LMV324 Rest: B/C/D als Folger auf GND, Versorgung +3V3"
- note added: "MAP (J2.58) — ratiometrisch 5 V → 0,625"
- note added: "O2 Schmalband (J2.38) — Folger an +3V3, Fallback (Breitband am CAN)"
- note added: "Senke gegen Klemmstrom-Pumpen der +3V3-Schiene (BAV199-Rückspeisung)"
- note added: "TPS (J2.49) — ratiometrisch 5 V → 0,625"
- note removed: "5v to 3.3v Opamp"
- note removed: "Baro Sensor"
- note removed: "Battery reference voltage"
- note removed: "Clutch Input"
- note removed: "Coolant Temperature Sensor"
- note removed: "Flex Sensor Input"
- note removed: "Inlet Air Temperature Sensor"
- note removed: "Map Sensor"
- note removed: "O2 Sensor"
- note removed: "Throttle Position Sensor"
- title: (none) -> Inputs
