File: hardware/ECU/Power-Regulator.kicad_sch (KiCad schematic)
At the start: 18 parts, among them U12 MC78M05_TO252

Commit message: Update ECU-Hardware, Dokumente und Explosionszeichnungen
Parts:
- removed C31, C33, C37: 0.1uF, Capacitor_SMD:C_0805_2012Metric, symbol Device:C
- removed C32, C34: 47uF, Capacitor_Tantalum_SMD:CP_EIA-3528-21_Kemet-B, symbol Device:CP
- removed C35, C36: 33uF, Capacitor_SMD:CP_Elec_6.3x7.7, symbol Device:CP
- removed D24: D_TVS, Diode_SMD:D_SMB, symbol Device:D_Zener
- removed D25: D_Schottky, Diode_SMD:D_SMA_Handsoldering, symbol Device:D_Schottky
- removed D26, D27, D28: LED, LED_SMD:LED_0805_2012Metric_Pad1.15x1.40mm_HandSolder, symbol Device:LED
- removed JP6: Jumper_2_Open, Jumper:SolderJumper-2_P1.3mm_Open_Pad1.0x1.5mm, symbol Jumper:Jumper_2_Open
- removed R67: 1k, Resistor_SMD:R_0805_2012Metric, symbol Device:R
- removed R68, R69: 470R, Resistor_SMD:R_0805_2012Metric, symbol Device:R
- removed U12: MC78M05_TO252, Package_TO_SOT_SMD:TO-252-2, symbol Regulator_Linear:MC78M05_TO252
- added C53, C54, C65, C73: 100nF/100V, Capacitor_SMD:C_1210_3225Metric, symbol Device:C
- added C55, C56: 4.7uF/100V, Capacitor_SMD:C_1210_3225Metric, symbol Device:C
- added C57: 1uF/50V, Capacitor_SMD:C_0805_2012Metric, symbol Device:C
- added C58, C63: 10uF/10V, Capacitor_SMD:C_0805_2012Metric, symbol Device:C
- added C59, C66: 100nF/25V, Capacitor_SMD:C_0805_2012Metric, symbol Device:C
- added C60: 39pF, Capacitor_SMD:C_0805_2012Metric, symbol Device:C
- added C61, C69: 100uF/50V, Capacitor_SMD:CP_Elec_8x10, symbol Device:CP
- added C62: 6800pF, Capacitor_SMD:C_0805_2012Metric, symbol Device:C
- added C64: 22uF/10V, Capacitor_SMD:C_1210_3225Metric, symbol Device:C
- added C67, C68, C74: 100nF, Capacitor_SMD:C_0805_2012Metric, symbol Device:C
- added C70, C72: 47uF/10V X7R, Capacitor_SMD:C_1210_3225Metric, symbol Device:C
- added C71: 10uF/50V X7R, Capacitor_SMD:C_1210_3225Metric, symbol Device:C
- added D41: SM8S24A, Rev3:D_DO-218AB, symbol Rev3:SM8S24A
- added D42: B560C, Diode_SMD:D_SMC, symbol Device:D_Schottky
- added D43, D44, D45: LED grn, LED_SMD:LED_0805_2012Metric, symbol Device:LED
- added IC5: LD1117S33, Package_TO_SOT_SMD:SOT-223-3_TabPin2, symbol Rev3:LD1117S33
- added L1: 10uH / 3.3A, Inductor_SMD:L_Bourns_SRR1260, symbol Device:L
- added L2: 8.2uH / 5A, Inductor_SMD:L_Bourns_SRR1260, symbol Device:L
- added Q6: SQM120N06-3M5L, Package_TO_SOT_SMD:TO-263-2, symbol Rev3:Q_NMOS_D2PAK
- added R114: 237k, Resistor_SMD:R_0805_2012Metric, symbol Device:R
- added R115: 56k2, Resistor_SMD:R_0805_2012Metric, symbol Device:R
- added R116: 162k, Resistor_SMD:R_0805_2012Metric, symbol Device:R
- added R117: 53k6, Resistor_SMD:R_0805_2012Metric, symbol Device:R
- added R118: 10k2, Resistor_SMD:R_0805_2012Metric, symbol Device:R
- added R119: 13k, Resistor_SMD:R_0805_2012Metric, symbol Device:R
- added R120: 470R, Resistor_SMD:R_0805_2012Metric, symbol Device:R
- added R121: 2k2, Resistor_SMD:R_0805_2012Metric, symbol Device:R
- added R122: 1k, Resistor_SMD:R_0805_2012Metric, symbol Device:R
- added U15: LM74700-Q1, Package_TO_SOT_SMD:SOT-23-6, symbol Rev3:LM74700-Q1
- added U16: TPS54360B-Q1, Package_SO:HSOP-8-1EP_3.9x4.9mm_P1.27mm_EP2.41x3.1mm_ThermalVias, symbol Rev3:TPS54360B-Q1
- added U17: TPS7B6950-Q1, Package_TO_SOT_SMD:SOT-223-3_TabPin2, symbol Rev3:TPS7B6950-Q1
- F2: value Polyfuse -> 3A / 63V; footprint Fuse:Fuse_0603_1608Metric -> Fuse:Fuse_1206_3216Metric; BOM Comments (none) -> 3A/65V flink 1206 (63V-Anforderung: 437er-Serie schafft nur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; Digikey Part Number 507-1817-1-ND -> 18-0483003.DRCT-ND; Manufacturer_Name Bel Fuse Inc. -> Littelfuse; Manufacturer_Part_Number 0ZCM0008FF2G -> 0483003.DR; Supplier (none) -> DigiKey; URL https://www.digikey.com.au/product-detail/en/bel-fuse-inc/0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 -> (none)
Connections:
- net +5V: now also C58.1, C70.1, C72.1, C74.1, IC5.3 (VIN), L2.2, R117.1, R122.1; no longer F2.1
- net 12V-PROT: now also C53.1, C55.1, C56.1, C57.1, C69.1, C71.1, C73.1, L1.2, R114.1, R121.1, U16.2 (VIN), U17.1 (IN)
- net 12V-SW: now also F2.1
- net GND: now also C53.2, C54.2, C55.2, C56.2, C57.2, C58.2, C59.2, C60.2, C61.2, C62.2, C63.2, C64.2, C65.2, C67.2, C68.2, C69.2, C70.2, C71.2, C72.2, C73.2, C74.2, D42.2 (A), D43.1 (K), D44.1 (K), D45.1 (K), IC5.1 (GND), R115.2, R116.2, R118.2, U15.2 (GND), U16.7 (GND), U16.9 (PAD), U17.2 (GND)
- net VDDA: now also C63.1, C67.1, U17.3 (OUT); no longer F2.2
- new net: C66.1, U16.1 (BOOT)
- new net: C66.2, D42.1 (K), L2.1, U16.8 (SW)
- new net: D45.2 (A), R122.2
- new net: D44.2 (A), R121.2
- new net: D43.2 (A), R120.2
- new net: C62.1, R119.2
- new net: C59.1, U15.1 (VCAP)
- new net +3V3: C64.1, C68.1, IC5.2 (VOUT), R120.1
- new net BUCK_COMP: C60.1, R119.1, U16.6 (COMP)
- new net BUCK_EN: R114.2, R115.1, U16.3 (EN)
- new net BUCK_FB: R117.2, R118.1, U16.5 (FB)
- new net BUCK_RT: R116.1, U16.4 (RT)
- new net ID_GATE: Q6.1 (G), U15.5 (GATE)
- new net PGND: D41.2
- new net VBAT_F: C54.1, F2.2, Q6.3 (S), U15.3 (EN), U15.6 (A)
- new net VBAT_ID: C61.1, C65.1, D41.1, L1.1, Q6.2 (D), U15.4 (K)
Other:
- note added: "1) EINGANGSSCHUTZ: 12V-SW -> Sicherung -> Ideal-Diode LM74700-Q1 (Verpolschutz, <20 mV) -> SM8S24A (Load Dump ISO 7637-2) -> Pi-Filter -> 12V-PROT"
- note added: "2) +5V HAUPTRAIL: TPS54360B-Q1 Buck, 600 kHz, UVLO 6,0 V ein / 5,2 V aus (Kurbel-Brownout-fest), Werte nach TI-Designbeispiel 5 V (SLVSDV1 Kap. 8.2)"
- note added: "3) VDDA SENSORVERSORGUNG: TPS7B6950-Q1 (5 V / 150 mA, kurzschlussfest, 40 V am Eingang). Speist J2.48 + NTC-Pullups; Polyfuse/TVS/10uF am Stecker (Conntectors)."
- note added: "4) +3V3 PERIPHERIE: LD1117S33 aus +5V, alleinige Quelle fuer MC33810-VDD, Flash, ADXL, MAX9926-Logik, LMV324, Watchdog, 74LVC1G125, BTF3050TE-VDD."
- note added: "EN = ANODE (immer ein). VCAP 100 nF lt. Datenblatt."
- note added: "Kompensation/RT/Boot/L/Cout = TI-Designbeispiel 5 V, 600 kHz (R4 13k, C5 6800p, C8 39p, L 8.2uH, Cout 2x47uF, B560C)."
- title: (none) -> Power Regulator
