File: hardware/ECU/knock-sensor.kicad_sch (KiCad schematic)
At the start: 4 parts, among them IC6 TPIC8101DW

Commit message: Update ECU-Hardware, Dokumente und Explosionszeichnungen
Parts:
- removed C38: 4700pF, Capacitor_SMD:C_0805_2012Metric, symbol Device:C
- removed C40: 2200 pF, Capacitor_SMD:C_0805_2012Metric, symbol Device:C
- added C75: 0.01uF, Capacitor_SMD:C_0805_2012Metric, symbol Device:C
- added C76, C78: CC0805KRX7R9BB104, Capacitor_SMD:C_0805_2012Metric, symbol Device:C
- added C77: 100nF, Capacitor_SMD:C_0805_2012Metric, symbol Device:C
- added C79: CC0805KKX7R7BB475, Capacitor_SMD:C_0805_2012Metric, symbol Device:C
- added C81, C82: CC0805JRX7R9BB332, Capacitor_SMD:C_0805_2012Metric, symbol Device:C
- added D46, D47: BAV199, Package_TO_SOT_SMD:SOT-23, symbol Diode:BAV199
- added IC6: 74AHCT125T14-13, Package_SO:TSSOP-14_4.4x5mm_P0.65mm, symbol KiCad-slef:74AHCT125T14-13
- added R123: 10k, Resistor_SMD:R_0805_2012Metric, symbol Device:R
- added R124: 1k, Resistor_SMD:R_0805_2012Metric, symbol Device:R
- added R125: 2k, Resistor_SMD:R_0805_2012Metric, symbol Device:R
- added R126, R131, R132: RC0805FR-071ML, Resistor_SMD:R_0805_2012Metric, symbol Device:R
- added R127, R128, R129, R130: RC0805FR-07100KL, Resistor_SMD:R_0805_2012Metric, symbol Device:R
- added U18: 74LVC1G125, Package_TO_SOT_SMD:SOT-353_SC-70-5, symbol Rev3:74LVC1G125
- added Y1: CSTCR4M00G53-R0, Crystal:Resonator_SMD_Murata_CSTCR_4.5x2x1.15mm, symbol Rev3:Resonator_3Pin
- C80: renamed from C39; value 0.022uF -> CC0805KRX7R9BB104; Capacity (none) -> 0.1uF; Digikey Part Number (none) -> 311-1140-1-ND; Height (none) -> 0.95; Manufacturer_Name YAGEO -> Yageo; Manufacturer_Part_Number CC0805KPX7R9BB223 -> CC0805KRX7R9BB104; Mouser Part Number (none) -> 603-CC805KRX7R9BB104; Mouser Price/Stock (none) -> https://www.mouser.co.uk/ProductDetail/YAGEO/CC0805KRX7R9BB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; Supplier (none) -> DigiKey; URL https://yageogroup.com/content/datasheet/asset/file/UPY-GPH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 -> (none)
- IC7: renamed from IC6; footprint SOIC127P1030X265-20N -> Package_SO:SOIC-20W_7.5x12.8mm_P1.27mm; Digikey Part Number (none) -> 296-15132-1-ND; Manufacturer_Part_Number TPIC8101DW -> TPIC8101DWR; Supplier (none) -> DigiKey
Connections:
- net GND: now also C75.1, C76.1, C77.2, C78.1, C79.1, D46.1 (A1), D47.1 (A1), IC6.1 (1~{OE}), IC6.10 (3~{OE}), IC6.13 (4~{OE}), IC6.4 (2~{OE}), IC6.7 (GND), R125.2, R131.1, R132.1, U18.3 (GND), Y1.2 (GND)
- net MCU-D37: now also IC6.2 (1A), R123.2, U18.1 (~{OE}); no longer IC7.8 (~{CS})
- net MISO: now also U18.4 (Y); no longer IC7.11 (SDO)
- net MOSI: now also IC6.5 (2A); no longer IC7.12 (SDI)
- net SCLK: now also IC6.12 (4A); no longer IC7.13 (SCLK)
- net at IC7.10 (XOUT): now also R126.2, Y1.3
- net CH2N: now reaches IC7.16 (CH2N)
- net CH2N: now also R128.1, R130.1
- net CH2FB: now reaches IC7.17 (CH2FB)
- net CH2FB: now also R128.2
- net CH1FB: now reaches IC7.18 (CH1FB)
- net CH1FB: now also R127.2
- net CH1N: now reaches IC7.19 (CH1N)
- net CH1N: now also R127.1, R129.1
- net Knock-OUT: now reaches IC7.4 (OUT)
- net Knock-OUT: now also R124.1
- net Knock-INT: now reaches IC7.7 (INT/HOLD)
- net Knock-INT: now also IC6.8 (3Y)
- net at IC7.9 (XIN): now also R126.1, Y1.1
- net VDD renamed +5V
- net +5V: now also C76.2, C78.2, C79.2, D46.2 (K2), D47.2 (K2), IC6.14 (VCC)
- net VREF-KS renamed CH1P
- new net: C81.1, R129.2
- new net: C82.1, R130.2
- new net +3V3: C77.1, R123.1, U18.5 (VCC)
- new net Knock-CS: IC6.3 (1Y), IC7.8 (~{CS})
- new net Knock-SCLK: IC6.11 (4Y), IC7.13 (SCLK)
- new net Knock-SDI: IC6.6 (2Y), IC7.12 (SDI)
- new net Knock-SDO: IC7.11 (SDO), U18.2 (A)
- new net Knock-Sensor-1: C81.2, D46.3 (K1A2), R131.2
- new net Knock-Sensor-2: C82.2, D47.3 (K1A2), R132.2
- new net MCU-A17: C75.2, R124.2, R125.1
- new net MCU-D36: IC6.9 (3A)
- no-connect marks 0 -> 3
Other:
- title: (none) -> Knock Sensor
- moved on the sheet: C80, IC7
