File: hardware/ECU/Drivers.kicad_sch (KiCad schematic)
At the start: 36 parts, among them Q2 ISL9V5036P3-F085, Q3 ISL9V5036P3-F085, Q4 ISL9V5036P3-F085, Q5 ISL9V5036P3-F085, SW3 SW_DPDT_x2, U6 TC4424A, U7 MC33810, U8 TC4424A

Commit message: Update ECU-Hardware, Dokumente und Explosionszeichnungen
Parts:
- removed C11: 1uF, Capacitor_SMD:C_0805_2012Metric, symbol Device:C
- removed C12: 0.1uF, Capacitor_SMD:C_0805_2012Metric, symbol Device:C
- removed D12, D13, D2, D3: LED, LED_SMD:LED_0805_2012Metric, symbol Device:LED
- removed F1: Polyfuse, Fuse:Fuse_1812_4532Metric, symbol Device:Polyfuse
- removed Q5: ISL9V5036P3-F085, TO254P470X1016X2019-3P, symbol ISL9V5036P3-F085:ISL9V5036P3-F085
- removed R10, R11, R21, R22: 33, Resistor_SMD:R_0805_2012Metric, symbol Device:R
- removed R12, R13, R19, R20: 1k, Resistor_SMD:R_0805_2012Metric, symbol Device:R
- removed R16: 10k, Resistor_SMD:R_0805_2012Metric, symbol Device:R
- removed SW3: SW_DPDT_x2, Misc:AYZ0202AGRLC, symbol Misc:AYZ0202AGRLC
- removed U6, U8: TC4424A, Package_SO:SOIC-8_3.9x4.9mm_P1.27mm, symbol IC_Automotive:TC4424A
- added C15, C17: 0.1uF, Capacitor_SMD:C_0805_2012Metric, symbol Device:C
- added C16, C18: 33uF, Capacitor_SMD:CP_Elec_6.3x7.7, symbol Device:CP
- added C19, C20: 100n, Capacitor_SMD:C_0805_2012Metric, symbol Device:C
- added Q1: ISL9V5036P3-F085, ISL9V5036P3-F085:TO254P470X1016X2019-3P, symbol ISL9V5036P3-F085:ISL9V5036P3-F085
- added R27, R31, R32, R33, R34, R35: 10k, Resistor_SMD:R_0805_2012Metric, symbol Device:R
- added R28, R29, R53, R54: 33, Resistor_SMD:R_0805_2012Metric, symbol Device:R
- added R30: 20m, Resistor_SMD:R_2512_6332Metric, symbol Device:R
- added R36, R37, R38, R39, R42, R43, R44, R45: 18k, Resistor_SMD:R_1206_3216Metric, symbol Device:R
- added R46, R47, R48, R49: 4.02k, Resistor_SMD:R_0805_2012Metric, symbol Device:R
- added R50: 100k, Resistor_SMD:R_0805_2012Metric, symbol Device:R
- added U8: TPS3823-33DBV, Package_TO_SOT_SMD:SOT-23-5, symbol Rev3:TPS3823-33
- added U9: 74LVC1G00, Package_TO_SOT_SMD:SOT-353_SC-70-5, symbol Rev3:74LVC1G00
- D10: renamed from D6; Supplier (none) -> DigiKey
- D11: renamed from D7; Supplier (none) -> DigiKey
- D12: renamed from D8; Supplier (none) -> DigiKey
- D13: renamed from D9; Supplier (none) -> DigiKey
- D14: renamed from D10; Digikey Part Number 475-1415-1-ND -> 160-1415-1-ND; Manufacturer_Name OSRAM -> Lite-On; Manufacturer_Part_Number LH R974-LP-1 -> LTST-C170KRKT; Supplier (none) -> DigiKey
- D15: renamed from D11; Digikey Part Number 475-1415-1-ND -> 160-1415-1-ND; Manufacturer_Name OSRAM -> Lite-On; Manufacturer_Part_Number LH R974-LP-1 -> LTST-C170KRKT; Supplier (none) -> DigiKey
- D8: renamed from D4; Digikey Part Number 475-1415-1-ND -> 160-1415-1-ND; Manufacturer_Name OSRAM -> Lite-On; Manufacturer_Part_Number LH R974-LP-1 -> LTST-C170KRKT; Supplier (none) -> DigiKey
- D9: renamed from D5; Digikey Part Number 475-1415-1-ND -> 160-1415-1-ND; Manufacturer_Name OSRAM -> Lite-On; Manufacturer_Part_Number LH R974-LP-1 -> LTST-C170KRKT; Supplier (none) -> DigiKey
- Q2, Q3, Q4: footprint TO254P470X1016X2019-3P -> ISL9V5036P3-F085:TO254P470X1016X2019-3P; Digikey Part Number (none) -> ISL9V5036P3-F085-ND; Supplier (none) -> DigiKey
- R40: renamed from R14; Supplier (none) -> DigiKey
- R41: renamed from R15; Supplier (none) -> DigiKey
- R51: renamed from R17; Supplier (none) -> DigiKey
- R52: renamed from R18; Supplier (none) -> DigiKey
- U7: BOM Comments (none) -> Last Time Buy 30.04.2027 - Bedarf sichern; Digikey Part Number (none) -> MCZ33810EK-ND; Supplier (none) -> DigiKey; now left out of the parts list
Connections:
- net +3V3: now also C15.2, C16.1, C19.1, C20.1, R27.2, R35.2, U8.3 (~{MR}), U8.5 (VDD), U9.5 (VCC)
- net GND: now also C15.1, C16.2, C17.2, C18.2, C19.2, C20.2, R50.2, U8.2 (GND), U9.3 (GND); no longer Q2.3, Q3.3, Q4.3, U7.33 (GND)
- net IGN1: now also R36.1
- net IGN2: now also Q1.2, R37.1; no longer Q3.2
- net IGN3: now also Q3.2, R38.1; no longer Q4.2
- net IGN4: now also Q4.2, R39.1
- net INJ1: now also D11.1 (K), U7.1 (OUT0); no longer D12.1 (K), U7.17 (OUT3)
- net INJ3: now also D13.1 (K), U7.32 (OUT2); no longer D11.1 (K), U7.1 (OUT0)
- net INJ4: now also D12.1 (K), U7.17 (OUT3); no longer D13.1 (K), U7.32 (OUT2)
- net MC33810_1-CS: now also R27.1
- net OUTEN_1: now also R35.1, U9.4 (Y)
- net G_IGN4: now reaches Q4.1
- net G_IGN4: now also R34.1, R54.1
- net G_IGN3: now reaches Q3.1
- net G_IGN3: now also R33.1, R53.1
- net T_IGN2: now reaches U7.14 (GD1)
- net T_IGN2: now also R28.2
- net T_IGN1: now reaches U7.3 (GD0)
- net T_IGN1: now also R29.2
- net T_IGN3: now reaches U7.30 (GD2)
- net T_IGN3: now also R53.2
- net T_IGN4: now reaches U7.19 (GD3)
- net T_IGN4: now also R54.2
- net G_IGN1: now reaches Q2.1
- net G_IGN1: now also R29.1, R31.1
- net FB1: now reaches U7.15 (FB1)
- net FB1: now also R43.2, R47.1
- net FB3: now reaches U7.18 (FB3)
- net FB3: now also R45.2, R49.1
- net FB0: now reaches U7.2 (FB0)
- net FB0: now also R42.2, R46.1
- net IGBT_E: now reaches U7.26 (RSP)
- net IGBT_E: now also Q2.3, Q3.3, Q4.3, Q1.3, R30.1, R31.2, R32.2, R33.2, R34.2
- net PGND: now reaches U7.27 (RSN)
- net PGND: now also U7.33 (GND), R30.2, R46.2, R47.2, R48.2, R49.2
- net FB2: now reaches U7.31 (FB2)
- net FB2: now also R44.2, R48.1
- net 12V-SW renamed 12V-PROT
- net 12V-PROT: now also C17.1, C18.1
- new net: R36.2, R42.1
- new net: R39.2, R45.1
- new net: R38.2, R44.1
- new net: R37.2, R43.1
- new net G_IGN2: Q1.1, R28.1, R32.1
- new net MCU-D2: R50.1, U9.1 (A)
- new net MCU-D3: U8.4 (WDI)
- new net WDT-RESET: U8.1 (~{RESET}), U9.2 (B)
- no-connect marks 0 -> 11
Other:
- note added: "Brownout/MCU-Absturz -> RESET low -> NAND=HIGH -> alle 8 Endstufen aus."
- note added: "Freigabe nur bei MCU-D2=HIGH UND Watchdog-RESET=HIGH (WDI<1.6s von MCU-D3)."
- note added: "OUTEN-Safety: OUTEN aktiv LOW, R16 Pull-Up +3V3 (Boot=AUS)."
- note added: "RSP=IGBT_E, RSN=PGND (Kelvin-Layout!), Schwellen per SPI-DAC, Gain=2"
- note added: "Rev 3.0: MC33810 GD0-3 (5-9V Ladungspumpe) -> 33R -> ISL9V5036 direkt."
- note added: "TC4424/SW3/F1/IGN_V+ entfallen. VPWR/Freilauf an 12V-PROT. U7-GND = PGND (Injektor-Rueckstrom)."
- note added: "Zuendstrom-Shunt: alle IGBT-Emitter -> 20mOhm -> PGND"
- title: (none) -> Ignition and Injector Driver

Commit message: new file:   hardware/ECU/.step 	modified:   hardware/ECU/Conntectors.kicad_sch 	modified:   hardware/ECU/Drivers.kicad_sch 	modified:   hardware/ECU/ECU.kicad_pcb 	modified:   hardware/ECU/ECU.kicad_pro 	modified:   hardware/ECU/ECU.kicad_sch 	modified:   hardware/ECU/output/ECU.csv 	deleted:    hardware/ECU/output/Pinout.xlsx 	new file:   hardware/ECU/output/gerber files/BOM-JLCPCB.csv 	deleted:    hardware/ECU/output/gerber files/ECU-PTH.drl 	new file:   hardware/ECU/output/gerber files/ECU-all-pos-JLCPCB.csv 	new file:   hardware/ECU/output/gerber files/ECU-all-pos.csv 	deleted:    hardware/ECU/output/gerber files/ECU-all.pos 	modified:   hardware/ECU/output/gerber files/ECU.csv 	renamed:    hardware/ECU/output/gerber files/ECU-B_Adhesive.gbr -> hardware/ECU/output/gerber files/gerber/ECU-B_Adhesive.gbr 	renamed:    hardware/ECU/output/gerber files/ECU-B_Courtyard.gbr -> hardware/ECU/output/gerber files/gerber/ECU-B_Courtyard.gbr 	renamed:    hardware/ECU/output/gerber files/ECU-B_Cu.gbr -> hardware/ECU/output/gerber files/gerber/ECU-B_Cu.gbr 	renamed:    hardware/ECU/output/gerber files/ECU-B_Fab.gbr -> hardware/ECU/output/gerber files/gerber/ECU-B_Fab.gbr 	renamed:    hardware/ECU/output/gerber files/ECU-B_Mask.gbr -> hardware/ECU/output/gerber files/gerber/ECU-B_Mask.gbr 	renamed:    hardware/ECU/output/gerber files/ECU-B_Paste.gbr -> hardware/ECU/output/gerber files/gerber/ECU-B_Paste.gbr 	renamed:    hardware/ECU/output/gerber files/ECU-B_Silkscreen.gbr -> hardware/ECU/output/gerber files/gerber/ECU-B_Silkscreen.gbr 	renamed:    hardware/ECU/output/gerber files/ECU-Edge_Cuts.gbr -> hardware/ECU/output/gerber files/gerber/ECU-Edge_Cuts.gbr 	renamed:    hardware/ECU/output/gerber files/ECU-F_Adhesive.gbr -> hardware/ECU/output/gerber files/gerber/ECU-F_Adhesive.gbr 	renamed:    hardware/ECU/output/gerber files/ECU-F_Courtyard.gbr -> hardware/ECU/output/gerber files/gerber/ECU-F_Courtyard.gbr 	renamed:    hardware/ECU/output/gerber files/ECU-F_Cu.gbr -> hardwar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
Parts:
- Q1, Q2, Q3, Q4: now left out of the parts list
Changed lines of the file:
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@@
 		(body_style 1)
 		(exclude_from_sim no)
-		(in_bom yes)
+		(in_bom no)
 		(on_board yes)
-		(in_pos_files yes)
+		(in_pos_files no)
 		(dnp no)
 		(property "Reference" "Q4"
@@
 		(body_style 1)
 		(exclude_from_sim no)
-		(in_bom yes)
+		(in_bom no)
 		(on_board yes)
-		(in_pos_files yes)
+		(in_pos_files no)
 		(dnp no)
 		(property "Reference" "Q1"
@@
 		(body_style 1)
 		(exclude_from_sim no)
-		(in_bom yes)
+		(in_bom no)
 		(on_board yes)
-		(in_pos_files yes)
+		(in_pos_files no)
 		(dnp no)
 		(property "Reference" "Q3"
@@
 		(body_style 1)
 		(exclude_from_sim no)
-		(in_bom yes)
+		(in_bom no)
 		(on_board yes)
-		(in_pos_files yes)
+		(in_pos_files no)
 		(dnp no)
 		(property "Reference" "Q2"
@@
 		(in_bom no)
 		(on_board yes)
-		(in_pos_files yes)
+		(in_pos_files no)
 		(dnp no)
 		(property "Reference" "U7"
