File: hardware/ECU/ECU.kicad_sch (KiCad schematic)
At the start: 4 parts, among them U1 Teensy4.1

Commit message: Update ECU-Hardware, Dokumente und Explosionszeichnungen
Parts:
- added C1: 100nF, Capacitor_SMD:C_0805_2012Metric, symbol Device:C
- added TP1: TP_PROGRAM, TestPoint:TestPoint_Pad_D1.5mm, symbol Connector:TestPoint
- added TP2: TP_ON_OFF, TestPoint:TestPoint_Pad_D1.5mm, symbol Connector:TestPoint
- BT1: value Battery_Cell -> ML2032; footprint 2999:BAT_2999 -> Battery:BatteryHolder_Keystone_3034_1x20mm; BOM Comments (none) -> SMD-Halter 20 mm (Keystone 3034); Zelle ML2032 separat: Jau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; Digikey Part Number 36-2999-ND -> 36-3034-ND; Manufacturer_Name Keystone -> Keystone Electronics; Manufacturer_Part_Number 2999 -> 3034; Supplier (none) -> DigiKey
- D1: Digikey Part Number (none) -> DFLS240-7DICT-ND; Manufacturer_Name (none) -> Diodes Incorporated; Manufacturer_Part_Number (none) -> DFLS240-7; Supplier (none) -> DigiKey
- R1: Supplier (none) -> DigiKey
- U1: Digikey Part Number (none) -> 1568-16771-ND; Manufacturer_Name (none) -> SparkFun (PJRC); Manufacturer_Part_Number (none) -> DEV-16771; Supplier (none) -> DigiKey; now left out of the parts list
Connections:
- net +3V3: now also D1.2 (A); no longer D1.1 (K), U1.15 (3V3), U1.46 (3V3), U1.51 (3V3)
- net GND: now also C1.2
- net USB D+: now also U1.67 (D+); no longer U1.57 (D+)
- net USB D-: now also U1.66 (D-); no longer U1.56 (D-)
- net at R1.2: now also D1.1 (K); no longer D1.2 (A)
- net MCU-D33: now reaches U1.25 (33_MCLK2)
- net MCU-D37: now reaches U1.29 (37_CS)
- net MC33814-CS renamed MCU-D2
- net PROG: no longer names the net of U1.53 (PROGRAM)
- net PROG: now also TP1.1
- net RESET: no longer names the net of U1.54 (ON_OFF)
- net RESET: now also TP2.1
- net USB 5V: no longer names the net of U1.55 (5V)
- net USB GND: no longer names the net of U1.58 (GND)
- net VDD renamed +5V
- new net T_3V3: C1.1, U1.15 (3V3), U1.46 (3V3), U1.51 (3V3)
- no-connect marks 0 -> 11
